File: speaker.kicad_sch (KiCad schematic)
At the start: 7 parts, among them U29 LM4990MM

Commit message: minor changes
- removed the power, ambient light sensing circuits.
- minor changes in the primary MCU pinout.
- USB connector moved to MCU sheet.
- ESD protection added.
- removed the test points from the individual sheets.
- Improved readability.
Parts:
- removed C36, C37: 1u, symbol Device:C
- removed C38: 0.39u, symbol Device:C
- removed LS1: 8R Speaker, symbol Device:Speaker
- removed R51, R52: 20K, symbol Device:R
- removed U29: LM4990MM, Package_SO:TSSOP-8_3x3mm_P0.65mm, symbol Amplifier_Audio:LM4990MM
