File: 4L_character_matrix.kicad_sch (KiCad schematic)
At the start: 12 parts, among them U22 SN74LVC244A, U23 SM411006N/15, U24 SN74LVC244A, U25 SM411006N/15, U26 SM411006N/15, U27 SM411006N/15

Commit message: power circuit added
- addition of power circuit
- added bypassing circuit
- new formatting of the schematic
- root schematic updated
Connections:
- net VDIS renamed VDL
Changed lines of the file:
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@@
 		)
 	)
-	(global_label "VDIS"
+	(global_label "VDL"
 		(shape input)
 		(at 113.03 113.03 0)
@@
 		)
 		(property "Intersheetrefs" "${INTERSHEET_REFS}"
-			(at 120.1881 113.03 0)
+			(at 119.4019 113.03 0)
 			(effects
 				(font
@@
 		)
 	)
-	(global_label "VDIS"
+	(global_label "VDL"
 		(shape input)
 		(at 53.34 113.03 0)
@@
 		)
 		(property "Intersheetrefs" "${INTERSHEET_REFS}"
-			(at 60.4981 113.03 0)
+			(at 59.7119 113.03 0)
 			(effects
 				(font
