File: secondary_mcu.kicad_sch (KiCad schematic)
At the start: 50 parts, among them J3 Conn_ST_STDC14, J4 USB_C_Receptacle, Q1 2SC4116, SW4 SW_Wuerth_450301014042, SW5 SW_Omron_B3U-1000P, SW6 SW_Omron_B3U-1000P, U10 STM32U575RGT6, U11 USBLC6-2P6, U9 W25Q256JV

Commit message: PCB routing
- low power trace routing completion
Parts:
- removed TP15: ADC, TestPoint:TestPoint_Pad_D1.0mm, symbol Connector:TestPoint
- removed TP16: DAC, TestPoint:TestPoint_Pad_D1.0mm, symbol Connector:TestPoint
- removed TP17: PWM, TestPoint:TestPoint_Pad_D1.0mm, symbol Connector:TestPoint
Other:
- moved on the sheet: TP14

Commit message: Major overhaul required
- Secondary MCU External clock to be included
- possible removal of colon drivers
- priority towards the end product over schematic
- high speed signals to be tuned like QSPI and USB
Parts:
- J4: footprint Connector_USB:USB_C_Receptacle_Molex_105450-0101 -> precision_clock:USB_C_Receptacle_Molex_105450-0101
Other:
- note added: "Without a External Clock USB won't work"
Changed lines of the file:
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@@
 		)
 	)
+	(text "Without a External Clock USB won't work"
+		(exclude_from_sim no)
+		(at 362.712 134.874 0)
+		(effects
+			(font
+				(size 2.54 2.54)
+				(thickness 0.3175)
+				(color 0 194 0 1)
+			)
+		)
+	)
 	(text "PCB Stackup SIG+GND, GND, PWR, SIG+GND to be followed"
 		(exclude_from_sim no)
@@
 			)
 		)
-		(property "Footprint" "Connector_USB:USB_C_Receptacle_Molex_105450-0101"
+		(property "Footprint" "precision_clock:USB_C_Receptacle_Molex_105450-0101"
 			(at 339.09 78.74 0)
 			(effects

Commit message: Primary MCU rerouting
Parts:
- removed C26: 100n, Capacitor_SMD:C_0402_1005Metric, symbol Device:C
- removed J4: USB_C_Receptacle, precision_clock:USB_C_Receptacle_Molex_105450-0101, symbol Connector:USB_C_Receptacle
- removed R18, R25, R26: 5.1K, Resistor_SMD:R_0402_1005Metric, symbol Device:R
- removed U11: USBLC6-2P6, Package_TO_SOT_SMD:SOT-666, symbol Power_Protection:USBLC6-2P6
- removed U9: W25Q256JV, Package_SO:SOIC-8_5.3x5.3mm_P1.27mm, symbol precision_clock:W25Q256JV
- renumbered C27 to C26, C28 to C27, C29 to C28, C30 to C29, C31 to C30, C32 to C31, C33 to C32, C35 to C33, C36 to C35, C37 to C36, D8 to D10, D9 to D11, D10 to D12, D6 to D8, D7 to D9, R19 to R18, R20 to R19, R21 to R20, R22 to R21, R23 to R22, R24 to R23, TP20 to TP10, TP21 to TP11, TP22 to TP12, TP23 to TP13, TP14 to TP7, TP18 to TP8, TP19 to TP9, U10 to U9
Connections:
- no-connect marks 15 -> 5
Other:
- note removed: "QSPI Flash 256Mb/32B 133MHz"
- note removed: "USB Connector"
- note removed: "Without a External Clock USB won't work"

Commit message: Secondary MCU rerouting
Parts:
- removed JP8: DAC, Jumper:SolderJumper-2_P1.3mm_Open_RoundedPad1.0x1.5mm, symbol Jumper:SolderJumper_2_Open
- removed TP7: HSE_OUT, TestPoint:TestPoint_Pad_D1.0mm, symbol Connector:TestPoint
- removed TP8: VFB_UP, TestPoint:TestPoint_Pad_D1.0mm, symbol Connector:TestPoint
- added D13, D14: ESDALC6V1-1U2, precision_clock:ST ESDALC6V1-1U2, symbol Diode:ESD5Zxx
- renumbered FB4 to FB3, JP7 to JP6, TP13 to TP10, TP9 to TP6, TP10 to TP7, TP11 to TP8, TP12 to TP9
Connections:
- net M1A0 is gone; now on net MCU.RX: U9.14 (PA0)
- net M1A1 is gone; now on net MCU.TX: U9.15 (PA1)
- net M1A6 is gone; now on net AG.INT: U9.57 (PB5)
- net M1A7 is gone; now on net AG.SCL: U9.58 (PB6)
- net M2A0 is gone; now on net AG.SDA: U9.59 (PB7)
- net M2A1 is gone; now on net TH.SCL: U9.61 (PB8)
- net M2A2 is gone; now on net TH.SDA: U9.62 (PB9)
- net M2K0 is gone; now on net USART_TX: U9.51 (PC10)
- net QSPI_CS is gone; now on net USART_RX: U9.52 (PC11)
- net QSPI_IO3 is gone; now on net PWM: U9.22 (PA6)
- net AG.INT: no longer U9.54 (PD2)
- net AG.SCL: no longer U9.8 (PC0)
- net AG.SDA: no longer U9.9 (PC1)
- net GND: now also D13.2 (A), D14.2 (A)
- net MCU.RX: no longer U9.42 (PA9)
- net MCU.TX: no longer U9.43 (PA10)
- net NRST: now also C36.1, SW6.1, D14.1 (K); no longer C34.1, D11.1 (K), SW5.1
- net PWM: no longer U9.36 (PB15)
- net SWDCLK: now also D11.1 (K); no longer D9.1 (K)
- net TH.SCL: no longer U9.34 (PB13)
- net TH.SDA: no longer U9.35 (PB14)
- net USART_RX: now reaches J3.13 (VCP_RX)
- net USART_RX: now also D13.1 (K)
- net USART_TX: now reaches J3.14 (VCP_TX)
- net USART_TX: now also D12.1 (K)
- net DAC renamed VFB_C
- net HSE_OUT: no longer names the net of U9.41 (PA8)
- removed net IN_1: C36.1, D12.1 (K), SW6.1, U9.6 (PH1)
- net M1A2: no longer names the net of U9.50 (PA15)
- net M1A3: no longer names the net of U9.28 (PB2)
- net M1A4: no longer names the net of U9.55 (PB3)
- net M1A5: no longer names the net of U9.56 (PB4)
- net M1K0: no longer names the net of U9.25 (PC5)
- net M1K1: no longer names the net of U9.37 (PC6)
- net M1K2: no longer names the net of U9.38 (PC7)
- net M1K3: no longer names the net of U9.39 (PC8)
- net M1K4: no longer names the net of U9.40 (PC9)
- net M2A3: no longer names the net of U9.29 (PB10)
- net M2A4: no longer names the net of U9.33 (PB12)
- net M2A5: no longer names the net of U9.10 (PC2)
- net M2A6: no longer names the net of U9.11 (PC3)
- net M2A7: no longer names the net of U9.24 (PC4)
- net M2K1: no longer names the net of U9.53 (PC12)
- net M2K2: no longer names the net of U9.2 (PC13)
- net M2K3: no longer names the net of U9.3 (PC14)
- net M2K4: no longer names the net of U9.4 (PC15)
- net QSPI_CLK: no longer names the net of U9.17 (PA3)
- net QSPI_IO0: no longer names the net of U9.27 (PB1)
- net QSPI_IO1: no longer names the net of U9.26 (PB0)
- net QSPI_IO2: no longer names the net of U9.23 (PA7)
- net USB_D+: no longer names the net of U9.45 (PA12)
- net USB_D-: no longer names the net of U9.44 (PA11)
- net VFB.UP renamed VFB_D
- new net IN: C34.1, D9.1 (K), SW5.1, U9.54 (PD2)
- no-connect marks 5 -> 9
Other:
- note added: "ESD Protection"
- note added: "EXTI5"
- note added: "I2C1"
- note added: "I2C4"
- note added: "STLINK-V3MINIE programmer to be used"
- note added: "TIM3"
- note added: "UART4"
- note removed: "EXTI1"
- note removed: "I2C2"
- note removed: "I2C3"
- note removed: "OSPI1"
- note removed: "TIM15"
- note removed: "USART1"
- note removed: "USB"
- moved on the sheet: JP6, TP10, TP6, TP7, TP8, TP9

Commit message: Secondary MCU rerouting
- Bank 2 completion
- OSC net completion
Connections:
- net M1K0: now reaches U9.33 (PB12)
- net M1K1: now reaches U9.34 (PB13)
- net M1K2: now reaches U9.35 (PB14)
- net M1K3: now reaches U9.36 (PB15)
- net M1K4: now reaches U9.37 (PC6)
- net M1A7: now reaches U9.38 (PC7)
- net M1A6: now reaches U9.39 (PC8)
- net M1A5: now reaches U9.40 (PC9)
- net M1A4: now reaches U9.41 (PA8)
- net M1A0: now reaches U9.42 (PA9)
- net M1A1: now reaches U9.43 (PA10)
- net M1A2: now reaches U9.44 (PA11)
- net M1A3: now reaches U9.45 (PA12)

Commit message: Secondary MCU complete
Connections:
- net M2K0: now reaches U9.2 (PC13)
- net M2A7: now reaches U9.23 (PA7)
- net M2A6: now reaches U9.24 (PC4)
- net M2A5: now reaches U9.25 (PC5)
- net M2A4: now reaches U9.26 (PB0)
- net M2A0: now reaches U9.27 (PB1)
- net M2A1: now reaches U9.28 (PB2)
- net M2A2: now reaches U9.29 (PB10)
- net M2K1: now reaches U9.3 (PC14)
- net M2K2: now reaches U9.4 (PC15)
- net M2K3: now reaches U9.8 (PC0)
- net M2K4: now reaches U9.9 (PC1)
Other:
- note removed: "GPIO"

Commit message: PCB routing
Parts:
- removed JP6: PWM, Jumper:SolderJumper-2_P1.3mm_Open_RoundedPad1.0x1.5mm, symbol Jumper:SolderJumper_2_Open
- removed SW4: SW_Wuerth_450301014042, Button_Switch_THT:SW_Slide-03_Wuerth-WS-SLTV_10x2.5x6.4_P2.54mm, symbol Switch:SW_Wuerth_450301014042
- added SW4: SW_ALPSALPINE, precision_clock:SW_ALPSALPINE, symbol precision_clock:SW_ALPSALPINE
- renumbered C26 to C28, C27 to C29, C28 to C30, C29 to C31, C30 to C32, C31 to C33, C32 to C34, C33 to C35, C34 to C36, C35 to C37, C36 to C38, TP9 to TP10, TP10 to TP11, TP6 to TP7, TP7 to TP8, TP8 to TP9
Connections:
- net +3.3V: now also SW4.1 (A)
- net GND: now also SW4.3 (B), SW4.4 (GND)
- net PWM: now also R21.1
- net at R18.2: now also SW4.2 (C)
- no-connect marks 9 -> 11

Commit message: Schematic changes
- signal for dots are removed.
- power supply upgraded to buck converters.
- individually addressable Colon LEDs.
- second millisecond dot separator signal is not connected.
- buzzer can now be connected to PWM or DAC outputs.
Parts:
- removed RV1: 10K, precision_clock:Bourns 3352T, symbol Device:R_Potentiometer
- added JP1, JP2: SolderJumper_2_Open, symbol Jumper:SolderJumper_2_Open
- added RV3: 100K, precision_clock:Bourns 3352T, symbol Device:R_Potentiometer
- renumbered C28 to C25, C29 to C26, C30 to C27, C31 to C28, C32 to C29, C33 to C30, C34 to C31, C35 to C32, C36 to C33, C37 to C34, C38 to C35, FB3 to FB2, R18 to R11, R19 to R12, R20 to R13, R21 to R14, R22 to R15, R23 to R16, TP7 to TP4, TP8 to TP5, TP9 to TP6, TP10 to TP7, TP11 to TP8, U9 to U7
Connections:
- net +3.3V: now also RV3.1
- net ADC: now also RV3.2
- net GND: now also RV3.3
- net PWM: now also JP1.1 (A); no longer R14.1
- net M2A3: now reaches U7.56 (PB4)
- net M1A7: no longer names the net of U7.38 (PC7)
- net M2A7: no longer names the net of U7.23 (PA7)
- net VFB_C renamed DAC
- net DAC: now also JP2.1 (A)
- net VFB_D: no longer names the net of U7.20 (PA4)
- new net: JP1.2 (B), JP2.2 (B), R14.1
- no-connect marks 11 -> 13
