File: clock_display.kicad_sch (KiCad schematic)
At the start: 28 parts, among them U11 SA15-11SURKWA, U12 SA15-11SURKWA, U13 SA15-11SURKWA, U14 SA15-11SURKWA, U15 SA15-11SURKWA, U26 SN74LVC244A, U31 SN74LVC244A, U36 SN74LVC244A, U7 SA15-11SURKWA

Commit message: updated power
Parts:
- removed C47: 100n, Capacitor_SMD:C_0402_1005Metric, symbol Device:C
- removed D16, D17, D18, D19: LED, LED_THT:LED_D5.0mm, symbol Device:LED
- removed R51, R52, R53, R54: 10R, Resistor_SMD:R_0603_1608Metric, symbol Device:R
- removed U36: SN74LVC244A, Package_SO:TSSOP-20_4.4x6.5mm_P0.65mm, symbol 74xx:74AHC244
- added R11, R23: 10R, Resistor_SMD:R_0603_1608Metric, symbol Device:R
- U11, U12, U13, U14, U15, U7: Mouser (none) -> 604-SA15-11SURKWA
Connections:
- net GND: now also R23.2
- net K7: now also R11.2, R23.1; no longer U26.9 (2Y3)
- new net: R11.1, U26.9 (2Y3)
- no-connect marks 4 -> 0
Other:
- note removed: "HH:mm separator"
- note removed: "HHmmSSsss Character matrix drivers"
- note removed: "mm:SS separator"
- moved on the sheet: C25, C26, C44, C45, R45, R46, R47, R48, R49, R50, U26, U31
