File: Primary MCU.kicad_sch (KiCad schematic)
At the start: 34 parts, among them J1 Conn_ST_STDC14, J2 USB_C_Receptacle, SW1 SW_ALPSALPINE, SW3 SW_Omron_B3U-1000P, U4 W25Q256JV, U5 STM32U575RGT6, U6 USBLC6-2P6, Y1 Q13MC14620002, Y2 ECS-TXO-2520MV

Commit message: Restructuring
Connections:
- net QSPI_CS: now also U5.52 (PC11); no longer U5.20 (PA4)
- net USART_RX: now also U5.43 (PA10); no longer U5.21 (PA5)
- net USART_TX: now also U5.42 (PA9); no longer U5.24 (PC4)
- net LS.INT: now reaches U5.10 (PC2)
- net AG.SCL: now reaches U5.29 (PB10)
- net AG.SDA: now reaches U5.35 (PB14)
- net AG.INT: now reaches U5.36 (PB15)
- net PWM: now reaches U5.41 (PA8)
- net ENC.A: now reaches U5.50 (PA15)
- net ENC.B: now reaches U5.55 (PB3)
- net ENC.C: now reaches U5.56 (PB4)
- net TH.SCL: now reaches U5.58 (PB6)
- net TH.SDA: now reaches U5.59 (PB7)
- net LS.SCL: now reaches U5.8 (PC0)
- net LS.SDA: now reaches U5.9 (PC1)
- new net DAC.COL: U5.21 (PA5)
- new net DAC.DIS: U5.20 (PA4)
- no-connect marks 16 -> 17
Other:
- note added: "DAC1"
- note added: "EXTI15"
- note added: "EXTI4"
- note added: "I2C1"
- note added: "I2C2"
- note added: "I2C3"
- note added: "Primary MCU"
- note added: "TIM1"
- note added: "TIM2"
- note added: "USART1"
- note removed: "Primary MCU STM32U575RGT6"
- note removed: "USART3"
- moved on the sheet: C24, D3, D4, D5, D6, D7, SW3

Commit message: Pin out completion
Parts:
- added R14, R15: 10K, symbol Device:R
Connections:
- net LS.SCL is gone; now on net AG.SCL: U5.8 (PC0)
- net LS.SDA is gone; now on net AG.SDA: U5.9 (PC1)
- net +3.3V: now also R14.1, R15.1
- net AG.INT: now also U5.10 (PC2); no longer U5.36 (PB15)
- net AG.SCL: now also R14.2; no longer U5.29 (PB10)
- net AG.SDA: now also R15.2; no longer U5.35 (PB14)
- net LS.INT: now also U5.11 (PC3); no longer U5.10 (PC2)
- net DIS13: now reaches U5.2 (PC13)
- net COL1: now reaches U5.24 (PC4)
- net COL2: now reaches U5.25 (PC5)
- net DIS0: now reaches U5.28 (PB2)
- net DIS7: now reaches U5.33 (PB12)
- net DIS8: now reaches U5.34 (PB13)
- net ENC3: now reaches U5.37 (PC6)
- net ENC4: now reaches U5.38 (PC7)
- net ENC5: now reaches U5.39 (PC8)
- net COL3: now reaches U5.40 (PC9)
- net DIS11: now reaches U5.51 (PC10)
- net DIS12: now reaches U5.53 (PC12)
- net COL0: now reaches U5.54 (PD2)
- net DIS1: now reaches U5.57 (PB5)
- net DIS4: now reaches U5.61 (PB8)
- net DIS5: now reaches U5.62 (PB9)
- net ENC.A renamed ENC0
- net ENC.B renamed ENC1
- net ENC.C renamed ENC2
- net TH.SCL renamed DIS2
- net TH.SDA renamed DIS3
- new net DIS10: U5.36 (PB15)
- new net DIS6: U5.29 (PB10)
- new net DIS9: U5.35 (PB14)
- no-connect marks 17 -> 16
Other:
- note added: "EXTI3"
- note added: "EXTI8"
- note added: "I2C Terminations"
- note added: "MCU"
- note added: "TIM3"
- note removed: "EXTI15"
- note removed: "I2C1"
- note removed: "I2C2"
- note removed: "Primary MCU"
- moved on the sheet: C24, D3, D4, D5, D6, D7, SW3, U5
