File: Temperature & Humidity Sensor.kicad_sch (KiCad schematic)
At the start: 4 parts, among them U10 HDC1080

Commit message: Pin out completion
Parts:
- removed R21, R22: 10K, Resistor_SMD:R_0402_1005Metric, symbol Device:R

Commit message: Removal of Colon LEDs
Parts:
- renumbered C40 to C26, U10 to U9
Changed lines of the file:
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@@
 		(dnp no)
 		(fields_autoplaced yes)
-		(property "Reference" "#PWR046"
+		(property "Reference" "#PWR066"
 			(at 120.65 83.82 0)
 			(effects
@@
 			(project "Precision Clock"
 				(path "/c9a8ff63-a0d1-4125-9dd1-40fb53daf536/cc882cab-fb20-4552-b867-43569dfc2d06"
-					(reference "#PWR046")
+					(reference "#PWR066")
 					(unit 1)
 				)
@@
 		(dnp no)
 		(fields_autoplaced yes)
-		(property "Reference" "C40"
+		(property "Reference" "C26"
 			(at 109.22 87.6299 0)
 			(effects
@@
 			(project "Precision Clock"
 				(path "/c9a8ff63-a0d1-4125-9dd1-40fb53daf536/cc882cab-fb20-4552-b867-43569dfc2d06"
-					(reference "C40")
+					(reference "C26")
 					(unit 1)
 				)
@@
 		(on_board yes)
 		(dnp no)
-		(property "Reference" "U10"
+		(property "Reference" "U9"
 			(at 114.3 104.14 0)
 			(effects
@@
 			(project "Precision Clock"
 				(path "/c9a8ff63-a0d1-4125-9dd1-40fb53daf536/cc882cab-fb20-4552-b867-43569dfc2d06"
-					(reference "U10")
+					(reference "U9")
 					(unit 1)
 				)
@@
 		(dnp no)
 		(fields_autoplaced yes)
-		(property "Reference" "#PWR075"
+		(property "Reference" "#PWR065"
 			(at 105.41 101.6 0)
 			(effects
@@
 			(project "Precision Clock"
 				(path "/c9a8ff63-a0d1-4125-9dd1-40fb53daf536/cc882cab-fb20-4552-b867-43569dfc2d06"
-					(reference "#PWR075")
+					(reference "#PWR065")
 					(unit 1)
 				)
@@
 		(dnp no)
 		(fields_autoplaced yes)
-		(property "Reference" "#PWR077"
+		(property "Reference" "#PWR067"
 			(at 120.65 125.73 0)
 			(effects
@@
 			(project "Precision Clock"
 				(path "/c9a8ff63-a0d1-4125-9dd1-40fb53daf536/cc882cab-fb20-4552-b867-43569dfc2d06"
-					(reference "#PWR077")
-					(unit 1)
-				)
+					(reference "#PWR067")
+					(unit 1)
+				)

Commit message: removal of sensors
Other:
- note added: "BME690 to be used here."
Changed lines of the file:
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@@
+		)
+	)
+	(text "BME690 to be used here."
+		(exclude_from_sim no)
+		(at 168.656 85.344 0)
+		(effects
+			(font
+				(size 1.27 1.27)
+			)
 		)
 	)
