File: MCU.kicad_sch (KiCad schematic)
At the start: 34 parts, among them J1 Conn_ST_STDC14, J2 USB_C_Receptacle, SW1 B3U-1100P, SW2 B3U-1100P, U3 W25Q256JV, U4 STM32U575RGT6, U5 USBLC6-2P6, Y1 Q13MC14620002, Y2 ECS-TXO-2520MV

Commit message: Power subsystem updated
Connections:
- net COL0 is gone; now on net DIS.EN: U4.10 (PC2)
- net COL2 is gone; now on net USART_TX: U4.24 (PC4)
- net COL3 is gone; now on net USART_RX: U4.25 (PC5)
- net +BATT: no longer U4.1 (VBAT)
- net DIS.EN: no longer U4.40 (PC9)
- net USART_RX: no longer U4.43 (PA10)
- net USART_TX: no longer U4.42 (PA9)
- net ADC renamed ALS
- net COL1: no longer names the net of U4.11 (PC3)
- net DIS0: no longer names the net of U4.28 (PB2)
- net DIS1: no longer names the net of U4.55 (PB3)
- net DIS10: no longer names the net of U4.34 (PB13)
- net DIS11: no longer names the net of U4.35 (PB14)
- net DIS12: no longer names the net of U4.36 (PB15)
- net DIS13: no longer names the net of U4.53 (PC12)
- net DIS2: no longer names the net of U4.56 (PB4)
- net DIS3: no longer names the net of U4.57 (PB5)
- net DIS4: no longer names the net of U4.58 (PB6)
- net DIS5: no longer names the net of U4.59 (PB7)
- net DIS6: no longer names the net of U4.61 (PB8)
- net DIS7: no longer names the net of U4.62 (PB9)
- net DIS8: no longer names the net of U4.29 (PB10)
- net DIS9: no longer names the net of U4.33 (PB12)
- net LED.EN: no longer names the net of U4.51 (PC10)
- net LED.FB: no longer names the net of U4.21 (PA5)
- net PWM renamed BZ
- new net MCU_RTC: U4.1 (VBAT)
- no-connect marks 18 -> 19
Other:
- note added: "GPIO"

Commit message: Verification
Parts:
- renumbered C8 to C10, C9 to C11, C10 to C12, C11 to C13, C12 to C14, C13 to C15, C14 to C16, C15 to C17, C16 to C18, C3 to C5, C4 to C6, C5 to C7, C6 to C8, C7 to C9, R1 to R6, R2 to R7, R3 to R8, R4 to R9

Commit message: display driver update
Parts:
- removed R8, R9: 5.1K, Resistor_SMD:R_0402_1005Metric, symbol Device:R
- added C35: 100n, Capacitor_SMD:C_0402_1005Metric, symbol Device:C
- R1: renamed from R6; value 5.1K -> 3.3K
- renumbered C5 to C1, C14 to C10, C15 to C11, C16 to C12, C17 to C13, C18 to C14, C6 to C2, C7 to C3, C8 to C4, C9 to C5, C10 to C6, C11 to C7, C12 to C8, C13 to C9, R7 to R2, U3 to U1, U4 to U2, U5 to U3
Connections:
- net DIS.FB is gone; now on net QSPI_CS: U2.20 (PA4)
- net GND: now also C35.2
- net QSPI_CS: no longer U2.52 (PC11)
- net USART_RX: now also U2.52 (PC11); no longer U2.25 (PC5)
- net USART_TX: now also U2.51 (PC10); no longer U2.24 (PC4)
- net VBUS: now also C35.1
- net DIS.EN: no longer names the net of U2.10 (PC2)
- no-connect marks 19 -> 20
Other:
- note added: "USART3"
- note removed: "DAC1"
- note removed: "GPIO"
- note removed: "USART1"

Commit message: Display Driver Completion
Parts:
- removed U3: USBLC6-2P6, Package_TO_SOT_SMD:SOT-666, symbol Power_Protection:USBLC6-2P6
- removed Y1: Q13MC14620002, Crystal:Crystal_SMD_SeikoEpson_MC146-4Pin_6.7x1.5mm, symbol Device:Crystal_GND23
- added C15: 330p, Capacitor_SMD:C_0402_1005Metric, symbol Device:C
- added D7: ESDA25P35-1U1M, Diode_SMD:ST_QFN-2L_1.6x1.0mm, symbol precision_clock:ESDA25P35-1U1M
- added U3: ECMF02-2AMX6, Package_DFN_QFN:ST_UQFN-6L_1.5x1.7mm_P0.5mm, symbol Power_Protection:ECMF02-2AMX6
- added Y1: Q13MC14620002, Crystal:Crystal_SMD_SeikoEpson_MC146-4Pin_6.7x1.5mm, symbol precision_clock:Q13MC14620002
- C16: renamed from C35; value 100n -> 330p
- R1: value 3.3K -> 10K
- renumbered C9 to C10, C10 to C11, C11 to C12, C12 to C13, C13 to C5, C5 to C6, C6 to C7, C7 to C8, C8 to C9, D5 to D1, D6 to D2, D1 to D3, D2 to D4, D3 to D5, D4 to D6
Connections:
- net CC1: now also C15.1
- net CC2: now also C16.1
- net GND: now also C15.2, D7.2 (A), U3.3 (GND)
- net OSC32_IN: now also Y1.1
- net OSC32_OUT: now also Y1.4 (3)
- net USB_D+: now also U3.5 (D-_out)
- net USB_D-: now also U3.6 (D+_out)
- net VBUS: now also D7.1 (K); no longer C16.1
- net at J2.A7 (D-), J2.B7 (D-): now also U3.1 (D+_in)
- net at J2.A6 (D+), J2.B6 (D+): now also U3.2 (D-_in)
- net SCL0: now reaches U2.28 (PB2)
- net SCL2: now reaches U2.29 (PB10)
- net SDI2: now reaches U2.33 (PB12)
- net SDO2: now reaches U2.34 (PB13)
- net LE2: now reaches U2.35 (PB14)
- net OE: now reaches U2.36 (PB15)
- net SDI0: now reaches U2.55 (PB3)
- net SDO0: now reaches U2.56 (PB4)
- net LE0: now reaches U2.57 (PB5)
- net SCL1: now reaches U2.58 (PB6)
- net SDI1: now reaches U2.59 (PB7)
- net SDO1: now reaches U2.61 (PB8)
- net LE1: now reaches U2.62 (PB9)
- net ENC0 renamed ENC_A
- net ENC1 renamed ENC_B
- net ENC2 renamed ENC_SW
- no-connect marks 20 -> 26
Other:
- note added: "GPIO"
- note added: "TIM15"
- moved on the sheet: C1, C16, C5, D1, D2, D3, D4, D5, D6, J1, J2, R1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

Commit message: PCB Routing
Parts:
- removed D7: ESDA25P35-1U1M, Diode_SMD:ST_QFN-2L_1.6x1.0mm, symbol precision_clock:ESDA25P35-1U1M
Other:
- moved on the sheet: C15, C16, R1

Commit message: PCB Routing
Parts:
- removed C15, C16: 330p, Capacitor_SMD:C_0402_1005Metric, symbol Device:C
- removed U3: ECMF02-2AMX6, Package_DFN_QFN:ST_UQFN-6L_1.5x1.7mm_P0.5mm, symbol Power_Protection:ECMF02-2AMX6
- added D8: ESDA6V1SC5, Package_TO_SOT_SMD:SOT-23-5, symbol Power_Protection:ESDA6V1SC5
Connections:
- net +BATT is gone; now on net MCU_RTC: C14.1
- net CC1: now also D8.1 (K)
- net CC2: now also D8.3 (K)
- net GND: now also D8.2 (A)
- net USB_D+: now also J2.A6 (D+), J2.B6 (D+), D8.5 (K)
- net USB_D-: now also J2.A7 (D-), J2.B7 (D-), D8.4 (K)
- no-connect marks 26 -> 25
Other:
- moved on the sheet: C1, C5, D1, D2, D3, D4, D5, D6, J1, J2, R1, R2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

Commit message: Footprints added
Parts:
- renumbered C11 to C10, C5 to C11, C6 to C5, C7 to C6, C8 to C7, C9 to C8, C10 to C9, D8 to D7
Connections:
- net CC1: now also D7.3 (K); no longer D7.1 (K)
- net CC2: now also D7.1 (K); no longer D7.3 (K)

Commit message: Major Changes
Parts:
- added D3: LED, precision_clock:LED_LiteON_LTST-C281KGKT, symbol Device:LED
- added R3, R4: 750R, Resistor_SMD:R_0402_1005Metric, symbol Device:R
- renumbered C9 to C10, C10 to C11, C11 to C9, D7 to D4, D3 to D5, D4 to D6, D5 to D7, D6 to D8
Connections:
- net GND: now also R3.2, R4.2
- net TP_OUT: now reaches U2.10 (PC2)
- net TP_OUT: now also D3.2 (A)
- net ENC_SW2: now reaches U2.40 (PC9)
- net ENC_SW renamed ENC_SW1
- new net: D3.1 (K), R3.1, R4.1
- no-connect marks 25 -> 23
Other:
- note added: "EXTI9"
- note added: "Pulse Per Second"
- note added: "Time Pulse Out"
- moved on the sheet: C9, D1, D2, D5, D6, D7, D8, R2, SW1, SW2
