File: User Inputs.kicad_sch (KiCad schematic)
At the start: 10 parts, among them SW3 RotaryEncoder_Switch

Commit message: Display Driver Completion
Parts:
- renumbered C28 to C31, C29 to C32, C30 to C33, R21 to R10, R22 to R11, R23 to R12, R24 to R13, R25 to R14, R20 to R9
Connections:
- net ENC0 renamed ENC_A
- net ENC1 renamed ENC_B
- net ENC2 renamed ENC_SW
Other:
- note added: "ESD Protection to be added here"
Changed lines of the file:
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@@
 	(title_block
 		(title "User Input")
-		(date "2026-02-04")
+		(date "2026-02-06")
 		(rev "v0.0")
 		(company "TJ71PL")
@@
 		(comment 4 "Final verification incomplete")
 	)
+	(bus_alias "INP_BUS"
+		(members "ENC_A" "ENC_B" "ENC_SW")
+	)
+	(text "ESD Protection to be added here"
+		(exclude_from_sim no)
+		(at 140.97 124.714 0)
+		(effects
+			(font
+				(size 1.27 1.27)
+				(italic yes)
+			)
+		)
+	)
+	(junction
+		(at 194.31 99.06)
+		(diameter 0)
+		(color 0 0 0 0)
+	)
+	(junction
+		(at 88.9 96.52)
+		(diameter 0)
+		(color 0 0 0 0)
+	)
+	(junction
+		(at 127 106.68)
+		(diameter 0)
+		(color 0 0 0 0)
+	)
 	(junction
 		(at 101.6 106.68)
@@
 	)
 	(junction
-		(at 194.31 99.06)
-		(diameter 0)
-		(color 0 0 0 0)
-	)
-	(junction
-		(at 127 106.68)
-		(diameter 0)
-		(color 0 0 0 0)
-	)
-	(junction
 		(at 171.45 99.06)
-		(diameter 0)
-		(color 0 0 0 0)
-	)
-	(junction
-		(at 88.9 96.52)
 		(diameter 0)
 		(color 0 0 0 0)
@@
 	(wire
 		(pts
+			(xy 194.31 99.06) (xy 209.55 99.06)
+		)
+		(stroke
+			(width 0)
+			(type default)
+		)
+	)
+	(wire
+		(pts
+			(xy 78.74 96.52) (xy 88.9 96.52)
+		)
+		(stroke
+			(width 0)
+			(type default)
+		)
+	)
+	(wire
+		(pts
 			(xy 101.6 109.22) (xy 101.6 106.68)
 		)
@@
 	(wire
 		(pts
+			(xy 78.74 106.68) (xy 101.6 106.68)
+		)
+		(stroke
+			(width 0)
+			(type default)
+		)
+	)
+	(wire
+		(pts
 			(xy 88.9 96.52) (xy 88.9 109.22)
 		)
@@
 	(wire
 		(pts
-			(xy 194.31 99.06) (xy 209.55 99.06)
-		)
-		(stroke
-			(width 0)
-			(type default)
-		)
-	)
-	(wire
-		(pts
 			(xy 120.65 106.68) (xy 127 106.68)
 		)
@@
 	(wire
 		(pts
-			(xy 78.74 96.52) (xy 88.9 96.52)
-		)
-		(stroke
-			(width 0)
-			(type default)
-		)
-	)
-	(wire
-		(pts
 			(xy 135.89 106.68) (xy 135.89 104.14)
 		)
@@
 		)
 	)
-	(wire
-		(pts
-			(xy 78.74 106.68) (xy 101.6 106.68)
-		)
-		(stroke
-			(width 0)
-			(type default)
-		)
-	)
 	(bus
 		(pts
@@
 		)
 	)
-	(label "ENC0"
-		(at 81.28 96.52 0)
+	(label "ENC_SW"
+		(at 199.39 99.06 0)
 		(effects
 			(font
@@
 		)
 	)
-	(label "ENC1"
-		(at 81.28 106.68 0)
+	(label "ENC_A"
+		(at 80.01 96.52 0)
 		(effects
 			(font
@@
 		)
 	)
-	(label "ENC2"
-		(at 200.66 99.06 0)
+	(label "ENC_B"
+		(at 80.01 106.68 0)
 		(effects
 			(font
@@
 		)
 	)
-	(hierarchical_label "ENC[0..2]"
+	(hierarchical_label "{INP_BUS}"
 		(shape output)
 		(at 73.66 93.98 180)
@@
 		)
 	)
-	(hierarchical_label "ENC[0..2]"
+	(hierarchical_label "{INP_BUS}"
 		(shape output)
 		(at 214.63 96.52 0)
@@
 		(dnp no)
 		(fields_autoplaced yes)
-		(property "Reference" "C28"
+		(property "Reference" "C31"
 			(at 92.71 111.7599 0)
 			(effects
@@
 			(project "Precision Clock"
 				(path "/c9a8ff63-a0d1-4125-9dd1-40fb53daf536/47769572-a111-4c65-a7b3-f0883fcb5fca"
-					(reference "C28")
+					(reference "C31")
 					(unit 1)
 				)
@@
 		(dnp no)
 		(fields_autoplaced yes)
-		(property "Reference" "R23"
+		(property "Reference" "R12"
 			(at 129.54 87.6299 0)
 			(effects
@@
 			(project "Precision Clock"
 				(path "/c9a8ff63-a0d1-4125-9dd1-40fb53daf536/47769572-a111-4c65-a7b3-f0883fcb5fca"
-					(reference "R23")
+					(reference "R12")
 					(unit 1)
 				)
@@
 		(dnp no)
 		(fields_autoplaced yes)
-		(property "Reference" "C29"
+		(property "Reference" "C32"
 			(at 105.41 111.7599 0)
 			(effects
@@
 			(project ""
 				(path "/c9a8ff63-a0d1-4125-9dd1-40fb53daf536/47769572-a111-4c65-a7b3-f0883fcb5fca"
-					(reference "C29")
+					(reference "C32")
 					(unit 1)
 				)
@@
 		(dnp no)
 		(fields_autoplaced yes)
-		(property "Reference" "#PWR080"
+		(property "Reference" "#PWR087"
 			(at 171.45 85.09 0)
 			(effects
@@
 			(project "Precision Clock"
 				(path "/c9a8ff63-a0d1-4125-9dd1-40fb53daf536/47769572-a111-4c65-a7b3-f0883fcb5fca"
-					(reference "#PWR080")
+					(reference "#PWR087")
 					(unit 1)
 				)
@@
 		(dnp no)
 		(fields_autoplaced yes)
-		(property "Reference" "#PWR078"
+		(property "Reference" "#PWR085"
 			(at 139.7 118.11 0)
 			(effects
@@
 			(project "Precision Clock"
 				(path "/c9a8ff63-a0d1-4125-9dd1-40fb53daf536/47769572-a111-4c65-a7b3-f0883fcb5fca"
-					(reference "#PWR078")
+					(reference "#PWR085")
 					(unit 1)
 				)
@@
 		(dnp no)
 		(fields_autoplaced yes)
-		(property "Reference" "R22"
+		(property "Reference" "R11"
 			(at 116.84 100.33 90)
 			(effects
@@
 			(project "Precision Clock"
 				(path "/c9a8ff63-a0d1-4125-9dd1-40fb53daf536/47769572-a111-4c65-a7b3-f0883fcb5fca"
-					(reference "R22")
+					(reference "R11")
 					(unit 1)
 				)
@@
 		(dnp no)
 		(fields_autoplaced yes)
-		(property "Reference" "#PWR081"
+		(property "Reference" "#PWR088"
 			(at 194.31 118.11 0)
 			(effects
@@
 			(project ""
 				(path "/c9a8ff63-a0d1-4125-9dd1-40fb53daf536/47769572-a111-4c65-a7b3-f0883fcb5fca"
-					(reference "#PWR081")
+					(reference "#PWR088")
 					(unit 1)
 				)
@@
 		(dnp no)
 		(fields_autoplaced yes)
-		(property "Reference" "R20"
+		(property "Reference" "R9"
 			(at 101.6 90.17 90)
 			(effects
@@
 			(project ""
 				(path "/c9a8ff63-a0d1-4125-9dd1-40fb53daf536/47769572-a111-4c65-a7b3-f0883fcb5fca"
-					(reference "R20")
+					(reference "R9")
 					(unit 1)
 				)
@@
 		(dnp no)
 		(fields_autoplaced yes)
-		(property "Reference" "#PWR074"
+		(property "Reference" "#PWR081"
 			(at 88.9 125.73 0)
 			(effects
@@
 			(project "Precision Clock"
 				(path "/c9a8ff63-a0d1-4125-9dd1-40fb53daf536/47769572-a111-4c65-a7b3-f0883fcb5fca"
-					(reference "#PWR074")
+					(reference "#PWR081")
 					(unit 1)
 				)
@@
 		(dnp no)
 		(fields_autoplaced yes)
-		(property "Reference" "R25"
+		(property "Reference" "R14"
 			(at 184.15 92.71 90)
 			(effects
@@
 			(project "Precision Clock"
 				(path "/c9a8ff63-a0d1-4125-9dd1-40fb53daf536/47769572-a111-4c65-a7b3-f0883fcb5fca"
-					(reference "R25")
+					(reference "R14")
 					(unit 1)
 				)
@@
 		(dnp no)
 		(fields_autoplaced yes)
-		(property "Reference" "C30"
+		(property "Reference" "C33"
 			(at 198.12 104.1399 0)
 			(effects
@@
 			(project "Precision Clock"
 				(path "/c9a8ff63-a0d1-4125-9dd1-40fb53daf536/47769572-a111-4c65-a7b3-f0883fcb5fca"
-					(reference "C30")
+					(reference "C33")
 					(unit 1)
 				)
@@
 		(dnp no)
 		(fields_autoplaced yes)
-		(property "Reference" "R24"
+		(property "Reference" "R13"
 			(at 173.99 87.6299 0)
 			(effects
@@
 			(project ""
 				(path "/c9a8ff63-a0d1-4125-9dd1-40fb53daf536/47769572-a111-4c65-a7b3-f0883fcb5fca"
-					(reference "R24")
+					(reference "R13")
 					(unit 1)
 				)
@@
 		(dnp no)
 		(fields_autoplaced yes)
-		(property "Reference" "#PWR076"
+		(property "Reference" "#PWR083"
 			(at 114.3 85.09 0)
 			(effects
@@
 			(project ""
 				(path "/c9a8ff63-a0d1-4125-9dd1-40fb53daf536/47769572-a111-4c65-a7b3-f0883fcb5fca"
-					(reference "#PWR076")
+					(reference "#PWR083")
 					(unit 1)
 				)
@@
 		(dnp no)
 		(fields_autoplaced yes)
-		(property "Reference" "R21"
+		(property "Reference" "R10"
 			(at 116.84 87.6299 0)
 			(effects
@@
 			(project "Precision Clock"
 				(path "/c9a8ff63-a0d1-4125-9dd1-40fb53daf536/47769572-a111-4c65-a7b3-f0883fcb5fca"
-					(reference "R21")
+					(reference "R10")
 					(unit 1)
 				)
@@
 		(on_board yes)
 		(dnp no)
-		(property "Reference" "#PWR077"
+		(property "Reference" "#PWR084"
 			(at 127 85.09 0)
 			(effects
@@
 			(project "Precision Clock"
 				(path "/c9a8ff63-a0d1-4125-9dd1-40fb53daf536/47769572-a111-4c65-a7b3-f0883fcb5fca"
-					(reference "#PWR077")
+					(reference "#PWR084")
 					(unit 1)
 				)
@@
 		(dnp no)
 		(fields_autoplaced yes)
-		(property "Reference" "#PWR079"
+		(property "Reference" "#PWR086"
 			(at 165.1 118.11 0)
 			(effects
@@
 			(project "Precision Clock"
 				(path "/c9a8ff63-a0d1-4125-9dd1-40fb53daf536/47769572-a111-4c65-a7b3-f0883fcb5fca"
-					(reference "#PWR079")
+					(reference "#PWR086")
 					(unit 1)
 				)
@@
 		(dnp no)
 		(fields_autoplaced yes)
-		(property "Reference" "#PWR075"
+		(property "Reference" "#PWR082"
 			(at 101.6 125.73 0)
 			(effects
@@
 			(project "Precision Clock"
 				(path "/c9a8ff63-a0d1-4125-9dd1-40fb53daf536/47769572-a111-4c65-a7b3-f0883fcb5fca"
-					(reference "#PWR075")
-					(unit 1)
-				)
+					(reference "#PWR082")
+					(unit 1)
+				)

Commit message: PCB Routing
Parts:
- renumbered C31 to C39, C32 to C40, C33 to C41
Changed lines of the file:
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@@
 		(dnp no)
 		(fields_autoplaced yes)
-		(property "Reference" "C31"
+		(property "Reference" "C39"
 			(at 92.71 111.7599 0)
 			(effects
@@
 			(project "Precision Clock"
 				(path "/c9a8ff63-a0d1-4125-9dd1-40fb53daf536/47769572-a111-4c65-a7b3-f0883fcb5fca"
-					(reference "C31")
+					(reference "C39")
 					(unit 1)
 				)
@@
 		(dnp no)
 		(fields_autoplaced yes)
-		(property "Reference" "C32"
+		(property "Reference" "C40"
 			(at 105.41 111.7599 0)
 			(effects
@@
 			(project ""
 				(path "/c9a8ff63-a0d1-4125-9dd1-40fb53daf536/47769572-a111-4c65-a7b3-f0883fcb5fca"
-					(reference "C32")
+					(reference "C40")
 					(unit 1)
 				)
@@
 		(dnp no)
 		(fields_autoplaced yes)
-		(property "Reference" "#PWR087"
+		(property "Reference" "#PWR096"
 			(at 171.45 85.09 0)
 			(effects
@@
 			(project "Precision Clock"
 				(path "/c9a8ff63-a0d1-4125-9dd1-40fb53daf536/47769572-a111-4c65-a7b3-f0883fcb5fca"
-					(reference "#PWR087")
+					(reference "#PWR096")
 					(unit 1)
 				)
@@
 		(dnp no)
 		(fields_autoplaced yes)
-		(property "Reference" "#PWR085"
+		(property "Reference" "#PWR094"
 			(at 139.7 118.11 0)
 			(effects
@@
 			(project "Precision Clock"
 				(path "/c9a8ff63-a0d1-4125-9dd1-40fb53daf536/47769572-a111-4c65-a7b3-f0883fcb5fca"
-					(reference "#PWR085")
+					(reference "#PWR094")
 					(unit 1)
 				)
@@
 		(dnp no)
 		(fields_autoplaced yes)
-		(property "Reference" "#PWR088"
+		(property "Reference" "#PWR097"
 			(at 194.31 118.11 0)
 			(effects
@@
 			(project ""
 				(path "/c9a8ff63-a0d1-4125-9dd1-40fb53daf536/47769572-a111-4c65-a7b3-f0883fcb5fca"
-					(reference "#PWR088")
+					(reference "#PWR097")
 					(unit 1)
 				)
@@
 		(dnp no)
 		(fields_autoplaced yes)
-		(property "Reference" "#PWR081"
+		(property "Reference" "#PWR090"
 			(at 88.9 125.73 0)
 			(effects
@@
 			(project "Precision Clock"
 				(path "/c9a8ff63-a0d1-4125-9dd1-40fb53daf536/47769572-a111-4c65-a7b3-f0883fcb5fca"
-					(reference "#PWR081")
+					(reference "#PWR090")
 					(unit 1)
 				)
@@
 		(dnp no)
 		(fields_autoplaced yes)
-		(property "Reference" "C33"
+		(property "Reference" "C41"
 			(at 198.12 104.1399 0)
 			(effects
@@
 			(project "Precision Clock"
 				(path "/c9a8ff63-a0d1-4125-9dd1-40fb53daf536/47769572-a111-4c65-a7b3-f0883fcb5fca"
-					(reference "C33")
+					(reference "C41")
 					(unit 1)
 				)
@@
 		(dnp no)
 		(fields_autoplaced yes)
-		(property "Reference" "#PWR083"
+		(property "Reference" "#PWR092"
 			(at 114.3 85.09 0)
 			(effects
@@
 			(project ""
 				(path "/c9a8ff63-a0d1-4125-9dd1-40fb53daf536/47769572-a111-4c65-a7b3-f0883fcb5fca"
-					(reference "#PWR083")
+					(reference "#PWR092")
 					(unit 1)
 				)
@@
 		(on_board yes)
 		(dnp no)
-		(property "Reference" "#PWR084"
+		(property "Reference" "#PWR093"
 			(at 127 85.09 0)
 			(effects
@@
 			(project "Precision Clock"
 				(path "/c9a8ff63-a0d1-4125-9dd1-40fb53daf536/47769572-a111-4c65-a7b3-f0883fcb5fca"
-					(reference "#PWR084")
+					(reference "#PWR093")
 					(unit 1)
 				)
@@
 		(dnp no)
 		(fields_autoplaced yes)
-		(property "Reference" "#PWR086"
+		(property "Reference" "#PWR095"
 			(at 165.1 118.11 0)
 			(effects
@@
 			(project "Precision Clock"
 				(path "/c9a8ff63-a0d1-4125-9dd1-40fb53daf536/47769572-a111-4c65-a7b3-f0883fcb5fca"
-					(reference "#PWR086")
+					(reference "#PWR095")
 					(unit 1)
 				)
@@
 		(dnp no)
 		(fields_autoplaced yes)
-		(property "Reference" "#PWR082"
+		(property "Reference" "#PWR091"
 			(at 101.6 125.73 0)
 			(effects
@@
 			(project "Precision Clock"
 				(path "/c9a8ff63-a0d1-4125-9dd1-40fb53daf536/47769572-a111-4c65-a7b3-f0883fcb5fca"
-					(reference "#PWR082")
-					(unit 1)
-				)
+					(reference "#PWR091")
+					(unit 1)
+				)

Commit message: Footprints added
Parts:
- renumbered C39 to C47, C40 to C48, C41 to C49, R9 to R20, R10 to R21, R11 to R22, R12 to R23, R13 to R24, R14 to R25
Changed lines of the file:
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@@
 		(dnp no)
 		(fields_autoplaced yes)
-		(property "Reference" "C39"
+		(property "Reference" "C47"
 			(at 92.71 111.7599 0)
 			(effects
@@
 			(project "Precision Clock"
 				(path "/c9a8ff63-a0d1-4125-9dd1-40fb53daf536/47769572-a111-4c65-a7b3-f0883fcb5fca"
-					(reference "C39")
+					(reference "C47")
 					(unit 1)
 				)
@@
 		(dnp no)
 		(fields_autoplaced yes)
-		(property "Reference" "R12"
+		(property "Reference" "R23"
 			(at 129.54 87.6299 0)
 			(effects
@@
 			(project "Precision Clock"
 				(path "/c9a8ff63-a0d1-4125-9dd1-40fb53daf536/47769572-a111-4c65-a7b3-f0883fcb5fca"
-					(reference "R12")
+					(reference "R23")
 					(unit 1)
 				)
@@
 		(dnp no)
 		(fields_autoplaced yes)
-		(property "Reference" "C40"
+		(property "Reference" "C48"
 			(at 105.41 111.7599 0)
 			(effects
@@
 			(project ""
 				(path "/c9a8ff63-a0d1-4125-9dd1-40fb53daf536/47769572-a111-4c65-a7b3-f0883fcb5fca"
-					(reference "C40")
+					(reference "C48")
 					(unit 1)
 				)
@@
 		(dnp no)
 		(fields_autoplaced yes)
-		(property "Reference" "#PWR096"
+		(property "Reference" "#PWR0118"
 			(at 171.45 85.09 0)
 			(effects
@@
 			(project "Precision Clock"
 				(path "/c9a8ff63-a0d1-4125-9dd1-40fb53daf536/47769572-a111-4c65-a7b3-f0883fcb5fca"
-					(reference "#PWR096")
+					(reference "#PWR0118")
 					(unit 1)
 				)
@@
 		(dnp no)
 		(fields_autoplaced yes)
-		(property "Reference" "#PWR094"
+		(property "Reference" "#PWR0116"
 			(at 139.7 118.11 0)
 			(effects
@@
 			(project "Precision Clock"
 				(path "/c9a8ff63-a0d1-4125-9dd1-40fb53daf536/47769572-a111-4c65-a7b3-f0883fcb5fca"
-					(reference "#PWR094")
+					(reference "#PWR0116")
 					(unit 1)
 				)
@@
 		(dnp no)
 		(fields_autoplaced yes)
-		(property "Reference" "R11"
+		(property "Reference" "R22"
 			(at 116.84 100.33 90)
 			(effects
@@
 			(project "Precision Clock"
 				(path "/c9a8ff63-a0d1-4125-9dd1-40fb53daf536/47769572-a111-4c65-a7b3-f0883fcb5fca"
-					(reference "R11")
+					(reference "R22")
 					(unit 1)
 				)
@@
 		(dnp no)
 		(fields_autoplaced yes)
-		(property "Reference" "#PWR097"
+		(property "Reference" "#PWR0119"
 			(at 194.31 118.11 0)
 			(effects
@@
 			(project ""
 				(path "/c9a8ff63-a0d1-4125-9dd1-40fb53daf536/47769572-a111-4c65-a7b3-f0883fcb5fca"
-					(reference "#PWR097")
+					(reference "#PWR0119")
 					(unit 1)
 				)
@@
 		(dnp no)
 		(fields_autoplaced yes)
-		(property "Reference" "R9"
+		(property "Reference" "R20"
 			(at 101.6 90.17 90)
 			(effects
@@
 			(project ""
 				(path "/c9a8ff63-a0d1-4125-9dd1-40fb53daf536/47769572-a111-4c65-a7b3-f0883fcb5fca"
-					(reference "R9")
+					(reference "R20")
 					(unit 1)
 				)
@@
 		(dnp no)
 		(fields_autoplaced yes)
-		(property "Reference" "#PWR090"
+		(property "Reference" "#PWR0112"
 			(at 88.9 125.73 0)
 			(effects
@@
 			(project "Precision Clock"
 				(path "/c9a8ff63-a0d1-4125-9dd1-40fb53daf536/47769572-a111-4c65-a7b3-f0883fcb5fca"
-					(reference "#PWR090")
+					(reference "#PWR0112")
 					(unit 1)
 				)
@@
 		(dnp no)
 		(fields_autoplaced yes)
-		(property "Reference" "R14"
+		(property "Reference" "R25"
 			(at 184.15 92.71 90)
 			(effects
@@
 			(project "Precision Clock"
 				(path "/c9a8ff63-a0d1-4125-9dd1-40fb53daf536/47769572-a111-4c65-a7b3-f0883fcb5fca"
-					(reference "R14")
+					(reference "R25")
 					(unit 1)
 				)
@@
 		(dnp no)
 		(fields_autoplaced yes)
-		(property "Reference" "C41"
+		(property "Reference" "C49"
 			(at 198.12 104.1399 0)
 			(effects
@@
 			(project "Precision Clock"
 				(path "/c9a8ff63-a0d1-4125-9dd1-40fb53daf536/47769572-a111-4c65-a7b3-f0883fcb5fca"
-					(reference "C41")
+					(reference "C49")
 					(unit 1)
 				)
@@
 		(dnp no)
 		(fields_autoplaced yes)
-		(property "Reference" "R13"
+		(property "Reference" "R24"
 			(at 173.99 87.6299 0)
 			(effects
@@
 			(project ""
 				(path "/c9a8ff63-a0d1-4125-9dd1-40fb53daf536/47769572-a111-4c65-a7b3-f0883fcb5fca"
-					(reference "R13")
+					(reference "R24")
 					(unit 1)
 				)
@@
 		(dnp no)
 		(fields_autoplaced yes)
-		(property "Reference" "#PWR092"
+		(property "Reference" "#PWR0114"
 			(at 114.3 85.09 0)
 			(effects
@@
 			(project ""
 				(path "/c9a8ff63-a0d1-4125-9dd1-40fb53daf536/47769572-a111-4c65-a7b3-f0883fcb5fca"
-					(reference "#PWR092")
+					(reference "#PWR0114")
 					(unit 1)
 				)
@@
 		(dnp no)
 		(fields_autoplaced yes)
-		(property "Reference" "R10"
+		(property "Reference" "R21"
 			(at 116.84 87.6299 0)
 			(effects
@@
 			(project "Precision Clock"
 				(path "/c9a8ff63-a0d1-4125-9dd1-40fb53daf536/47769572-a111-4c65-a7b3-f0883fcb5fca"
-					(reference "R10")
+					(reference "R21")
 					(unit 1)
 				)
@@
 		(on_board yes)
 		(dnp no)
-		(property "Reference" "#PWR093"
+		(property "Reference" "#PWR0115"
 			(at 127 85.09 0)
 			(effects
@@
 			(project "Precision Clock"
 				(path "/c9a8ff63-a0d1-4125-9dd1-40fb53daf536/47769572-a111-4c65-a7b3-f0883fcb5fca"
-					(reference "#PWR093")
+					(reference "#PWR0115")
 					(unit 1)
 				)
@@
 		(dnp no)
 		(fields_autoplaced yes)
-		(property "Reference" "#PWR095"
+		(property "Reference" "#PWR0117"
 			(at 165.1 118.11 0)
 			(effects
@@
 			(project "Precision Clock"
 				(path "/c9a8ff63-a0d1-4125-9dd1-40fb53daf536/47769572-a111-4c65-a7b3-f0883fcb5fca"
-					(reference "#PWR095")
+					(reference "#PWR0117")
 					(unit 1)
 				)
@@
 		(dnp no)
 		(fields_autoplaced yes)
-		(property "Reference" "#PWR091"
+		(property "Reference" "#PWR0113"
 			(at 101.6 125.73 0)
 			(effects
@@
 			(project "Precision Clock"
 				(path "/c9a8ff63-a0d1-4125-9dd1-40fb53daf536/47769572-a111-4c65-a7b3-f0883fcb5fca"
-					(reference "#PWR091")
-					(unit 1)
-				)
+					(reference "#PWR0113")
+					(unit 1)
+				)
