File: User Inputs.kicad_sch (KiCad schematic)
At the start: 10 parts, among them SW3 RotaryEncoder_Switch

Commit message: PCB Routing
Parts:
- renumbered C47 to C41, C48 to C42, C49 to C43, R20 to R22, R21 to R23, R22 to R24, R23 to R25, R24 to R26, R25 to R27
Changed lines of the file:
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@@
 		(dnp no)
 		(fields_autoplaced yes)
-		(property "Reference" "C47"
+		(property "Reference" "C41"
 			(at 92.71 111.7599 0)
 			(effects
@@
 			(project "Precision Clock"
 				(path "/c9a8ff63-a0d1-4125-9dd1-40fb53daf536/47769572-a111-4c65-a7b3-f0883fcb5fca"
-					(reference "C47")
+					(reference "C41")
 					(unit 1)
 				)
@@
 		(dnp no)
 		(fields_autoplaced yes)
-		(property "Reference" "R23"
+		(property "Reference" "R25"
 			(at 129.54 87.6299 0)
 			(effects
@@
 			(project "Precision Clock"
 				(path "/c9a8ff63-a0d1-4125-9dd1-40fb53daf536/47769572-a111-4c65-a7b3-f0883fcb5fca"
-					(reference "R23")
+					(reference "R25")
 					(unit 1)
 				)
@@
 		(dnp no)
 		(fields_autoplaced yes)
-		(property "Reference" "C48"
+		(property "Reference" "C42"
 			(at 105.41 111.7599 0)
 			(effects
@@
 			(project ""
 				(path "/c9a8ff63-a0d1-4125-9dd1-40fb53daf536/47769572-a111-4c65-a7b3-f0883fcb5fca"
-					(reference "C48")
+					(reference "C42")
 					(unit 1)
 				)
@@
 		(dnp no)
 		(fields_autoplaced yes)
-		(property "Reference" "#PWR0118"
+		(property "Reference" "#PWR0114"
 			(at 171.45 85.09 0)
 			(effects
@@
 			(project "Precision Clock"
 				(path "/c9a8ff63-a0d1-4125-9dd1-40fb53daf536/47769572-a111-4c65-a7b3-f0883fcb5fca"
-					(reference "#PWR0118")
+					(reference "#PWR0114")
 					(unit 1)
 				)
@@
 		(dnp no)
 		(fields_autoplaced yes)
-		(property "Reference" "#PWR0116"
+		(property "Reference" "#PWR0112"
 			(at 139.7 118.11 0)
 			(effects
@@
 			(project "Precision Clock"
 				(path "/c9a8ff63-a0d1-4125-9dd1-40fb53daf536/47769572-a111-4c65-a7b3-f0883fcb5fca"
-					(reference "#PWR0116")
+					(reference "#PWR0112")
 					(unit 1)
 				)
@@
 		(dnp no)
 		(fields_autoplaced yes)
-		(property "Reference" "R22"
+		(property "Reference" "R24"
 			(at 116.84 100.33 90)
 			(effects
@@
 			(project "Precision Clock"
 				(path "/c9a8ff63-a0d1-4125-9dd1-40fb53daf536/47769572-a111-4c65-a7b3-f0883fcb5fca"
-					(reference "R22")
+					(reference "R24")
 					(unit 1)
 				)
@@
 		(dnp no)
 		(fields_autoplaced yes)
-		(property "Reference" "#PWR0119"
+		(property "Reference" "#PWR0115"
 			(at 194.31 118.11 0)
 			(effects
@@
 			(project ""
 				(path "/c9a8ff63-a0d1-4125-9dd1-40fb53daf536/47769572-a111-4c65-a7b3-f0883fcb5fca"
-					(reference "#PWR0119")
+					(reference "#PWR0115")
 					(unit 1)
 				)
@@
 		(dnp no)
 		(fields_autoplaced yes)
-		(property "Reference" "R20"
+		(property "Reference" "R22"
 			(at 101.6 90.17 90)
 			(effects
@@
 			(project ""
 				(path "/c9a8ff63-a0d1-4125-9dd1-40fb53daf536/47769572-a111-4c65-a7b3-f0883fcb5fca"
-					(reference "R20")
+					(reference "R22")
 					(unit 1)
 				)
@@
 		(dnp no)
 		(fields_autoplaced yes)
-		(property "Reference" "#PWR0112"
+		(property "Reference" "#PWR0108"
 			(at 88.9 125.73 0)
 			(effects
@@
 			(project "Precision Clock"
 				(path "/c9a8ff63-a0d1-4125-9dd1-40fb53daf536/47769572-a111-4c65-a7b3-f0883fcb5fca"
-					(reference "#PWR0112")
+					(reference "#PWR0108")
 					(unit 1)
 				)
@@
 		(dnp no)
 		(fields_autoplaced yes)
-		(property "Reference" "R25"
+		(property "Reference" "R27"
 			(at 184.15 92.71 90)
 			(effects
@@
 			(project "Precision Clock"
 				(path "/c9a8ff63-a0d1-4125-9dd1-40fb53daf536/47769572-a111-4c65-a7b3-f0883fcb5fca"
-					(reference "R25")
+					(reference "R27")
 					(unit 1)
 				)
@@
 		(dnp no)
 		(fields_autoplaced yes)
-		(property "Reference" "C49"
+		(property "Reference" "C43"
 			(at 198.12 104.1399 0)
 			(effects
@@
 			(project "Precision Clock"
 				(path "/c9a8ff63-a0d1-4125-9dd1-40fb53daf536/47769572-a111-4c65-a7b3-f0883fcb5fca"
-					(reference "C49")
+					(reference "C43")
 					(unit 1)
 				)
@@
 		(dnp no)
 		(fields_autoplaced yes)
-		(property "Reference" "R24"
+		(property "Reference" "R26"
 			(at 173.99 87.6299 0)
 			(effects
@@
 			(project ""
 				(path "/c9a8ff63-a0d1-4125-9dd1-40fb53daf536/47769572-a111-4c65-a7b3-f0883fcb5fca"
-					(reference "R24")
+					(reference "R26")
 					(unit 1)
 				)
@@
 		(dnp no)
 		(fields_autoplaced yes)
-		(property "Reference" "#PWR0114"
+		(property "Reference" "#PWR0110"
 			(at 114.3 85.09 0)
 			(effects
@@
 			(project ""
 				(path "/c9a8ff63-a0d1-4125-9dd1-40fb53daf536/47769572-a111-4c65-a7b3-f0883fcb5fca"
-					(reference "#PWR0114")
+					(reference "#PWR0110")
 					(unit 1)
 				)
@@
 		(dnp no)
 		(fields_autoplaced yes)
-		(property "Reference" "R21"
+		(property "Reference" "R23"
 			(at 116.84 87.6299 0)
 			(effects
@@
 			(project "Precision Clock"
 				(path "/c9a8ff63-a0d1-4125-9dd1-40fb53daf536/47769572-a111-4c65-a7b3-f0883fcb5fca"
-					(reference "R21")
+					(reference "R23")
 					(unit 1)
 				)
@@
 		(on_board yes)
 		(dnp no)
-		(property "Reference" "#PWR0115"
+		(property "Reference" "#PWR0111"
 			(at 127 85.09 0)
 			(effects
@@
 			(project "Precision Clock"
 				(path "/c9a8ff63-a0d1-4125-9dd1-40fb53daf536/47769572-a111-4c65-a7b3-f0883fcb5fca"
-					(reference "#PWR0115")
+					(reference "#PWR0111")
 					(unit 1)
 				)
@@
 		(dnp no)
 		(fields_autoplaced yes)
-		(property "Reference" "#PWR0117"
+		(property "Reference" "#PWR0113"
 			(at 165.1 118.11 0)
 			(effects
@@
 			(project "Precision Clock"
 				(path "/c9a8ff63-a0d1-4125-9dd1-40fb53daf536/47769572-a111-4c65-a7b3-f0883fcb5fca"
-					(reference "#PWR0117")
+					(reference "#PWR0113")
 					(unit 1)
 				)
@@
 		(dnp no)
 		(fields_autoplaced yes)
-		(property "Reference" "#PWR0113"
+		(property "Reference" "#PWR0109"
 			(at 101.6 125.73 0)
 			(effects
@@
 			(project "Precision Clock"
 				(path "/c9a8ff63-a0d1-4125-9dd1-40fb53daf536/47769572-a111-4c65-a7b3-f0883fcb5fca"
-					(reference "#PWR0113")
-					(unit 1)
-				)
+					(reference "#PWR0109")
+					(unit 1)
+				)

Commit message: Major Changes
Parts:
- added C44: 10n, Capacitor_SMD:C_0402_1005Metric, symbol Device:C
- added D13, D14, D15, D16: ESDALC6V1-1U2, precision_clock:ST ESDALC6V1-1U2, symbol Diode:ESD5Zxx
- added R27, R29: 10K, Resistor_SMD:R_0402_1005Metric, symbol Device:R
- added SW4: PEC09-2320F-S0015, Rotary_Encoder:RotaryEncoder_Bourns_Horizontal_PEC09-2xxxF-Sxxxx, symbol Device:RotaryEncoder_Switch
- SW3: value RotaryEncoder_Switch -> PEC09-2320F-S0015; footprint (none) -> Rotary_Encoder:RotaryEncoder_Bourns_Horizontal_PEC09-2xxxF-Sxxxx; Mouser (none) -> 652-PEC092320FS0015
- renumbered R24 to R23, R23 to R24, R27 to R28
Connections:
- net +3.3V: now also R27.1
- net ENC_A: now also D13.1 (K)
- net ENC_B: now also D14.1 (K)
- net GND: now also C44.2, D13.2 (A), D14.2 (A), D15.2 (A), D16.2 (A), SW4.S2
- net ENC_SW renamed ENC_SW1
- net ENC_SW1: now also D15.1 (K)
- new net: R27.2, R29.1, SW4.S1
- new net ENC_SW2: C44.1, D16.1 (K), R29.2
- no-connect marks 0 -> 3
Other:
- note added: "User Input"
- note removed: "ESD Protection to be added here"
- moved on the sheet: C41, C42, C43, R22, R23, R24, R25, R26, R28

Commit message: Verification
Parts:
- SW1: renamed from SW4; value PEC09-2320F-S0015 -> PEC09-2320F-T0015; footprint Rotary_Encoder:RotaryEncoder_Bourns_Horizontal_PEC09-2xxxF-Sxxxx -> precision_clock:RotaryEncoder_Bourns_Horizontal_PEC09-2xxxF-Txxxx; Mouser 652-PEC092320FS0015 -> 652-PEC092320FT0015
- SW4: renamed from SW3; value PEC09-2320F-S0015 -> PEC09-2320F-T0015; footprint Rotary_Encoder:RotaryEncoder_Bourns_Horizontal_PEC09-2xxxF-Sxxxx -> precision_clock:RotaryEncoder_Bourns_Horizontal_PEC09-2xxxF-Txxxx; Mouser 652-PEC092320FS0015 -> 652-PEC092320FT0015
- renumbered C43 to C30, C41 to C31, C42 to C32, C44 to C33, D16 to D14, D14 to D15, D15 to D16, R28 to R25, R25 to R26, R23 to R27, R29 to R28, R27 to R29, R22 to R30, R26 to R31, R24 to R32
Other:
- note added: "30 Detents (15 pulses) 1.5mm Switch Stroke length"
- moved on the sheet: R25, R26, R27, R28, R29, R30, R31, R32, SW1, SW4

Commit message: Encoder placement
Parts:
- renumbered C32 to C30, C33 to C31, C31 to C32, C30 to C33, D15 to D13, D16 to D14, D14 to D15, D13 to D16, R27 to R25, R28 to R26, R26 to R27, R31 to R28, R32 to R29, R29 to R31, R25 to R32
Changed lines of the file:
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@@
 		(dnp no)
 		(fields_autoplaced yes)
-		(property "Reference" "C31"
+		(property "Reference" "C32"
 			(at 232.41 60.9599 0)
 			(effects
@@
 			(project "Precision Clock"
 				(path "/c9a8ff63-a0d1-4125-9dd1-40fb53daf536/47769572-a111-4c65-a7b3-f0883fcb5fca"
-					(reference "C31")
+					(reference "C32")
 					(unit 1)
 				)
@@
 		(dnp no)
 		(fields_autoplaced yes)
-		(property "Reference" "R26"
+		(property "Reference" "R27"
 			(at 92.71 85.0901 0)
 			(effects
@@
 			(project "Precision Clock"
 				(path "/c9a8ff63-a0d1-4125-9dd1-40fb53daf536/47769572-a111-4c65-a7b3-f0883fcb5fca"
-					(reference "R26")
+					(reference "R27")
 					(unit 1)
 				)
@@
 		(on_board yes)
 		(dnp no)
-		(property "Reference" "D15"
+		(property "Reference" "D13"
 			(at 207.518 85.344 90)
 			(effects
@@
 			(project "Precision Clock"
 				(path "/c9a8ff63-a0d1-4125-9dd1-40fb53daf536/47769572-a111-4c65-a7b3-f0883fcb5fca"
-					(reference "D15")
+					(reference "D13")
 					(unit 1)
 				)
@@
 		(dnp no)
 		(fields_autoplaced yes)
-		(property "Reference" "C32"
+		(property "Reference" "C30"
 			(at 232.41 86.3599 0)
 			(effects
@@
 			(project ""
 				(path "/c9a8ff63-a0d1-4125-9dd1-40fb53daf536/47769572-a111-4c65-a7b3-f0883fcb5fca"
-					(reference "C32")
+					(reference "C30")
 					(unit 1)
 				)
@@
 		(dnp no)
 		(fields_autoplaced yes)
-		(property "Reference" "C33"
+		(property "Reference" "C31"
 			(at 232.41 138.4299 0)
 			(effects
@@
 			(project "Precision Clock"
 				(path "/c9a8ff63-a0d1-4125-9dd1-40fb53daf536/47769572-a111-4c65-a7b3-f0883fcb5fca"
-					(reference "C33")
+					(reference "C31")
 					(unit 1)
 				)
@@
 		(dnp no)
 		(fields_autoplaced yes)
-		(property "Reference" "R27"
+		(property "Reference" "R25"
 			(at 82.55 69.85 90)
 			(effects
@@
 			(project "Precision Clock"
 				(path "/c9a8ff63-a0d1-4125-9dd1-40fb53daf536/47769572-a111-4c65-a7b3-f0883fcb5fca"
-					(reference "R27")
+					(reference "R25")
 					(unit 1)
 				)
@@
 		(dnp no)
 		(fields_autoplaced yes)
-		(property "Reference" "R29"
+		(property "Reference" "R31"
 			(at 138.43 107.9499 0)
 			(effects
@@
 			(project "Precision Clock"
 				(path "/c9a8ff63-a0d1-4125-9dd1-40fb53daf536/47769572-a111-4c65-a7b3-f0883fcb5fca"
-					(reference "R29")
+					(reference "R31")
 					(unit 1)
 				)
@@
 		(on_board yes)
 		(dnp no)
-		(property "Reference" "D16"
+		(property "Reference" "D14"
 			(at 207.518 110.744 90)
 			(effects
@@
 			(project "Precision Clock"
 				(path "/c9a8ff63-a0d1-4125-9dd1-40fb53daf536/47769572-a111-4c65-a7b3-f0883fcb5fca"
-					(reference "D16")
+					(reference "D14")
 					(unit 1)
 				)
@@
 		(dnp no)
 		(fields_autoplaced yes)
-		(property "Reference" "R25"
+		(property "Reference" "R32"
 			(at 146.05 62.23 90)
 			(effects
@@
 			(project "Precision Clock"
 				(path "/c9a8ff63-a0d1-4125-9dd1-40fb53daf536/47769572-a111-4c65-a7b3-f0883fcb5fca"
-					(reference "R25")
+					(reference "R32")
 					(unit 1)
 				)
@@
 		(on_board yes)
 		(dnp no)
-		(property "Reference" "D14"
+		(property "Reference" "D15"
 			(at 207.518 137.414 90)
 			(effects
@@
 			(project "Precision Clock"
 				(path "/c9a8ff63-a0d1-4125-9dd1-40fb53daf536/47769572-a111-4c65-a7b3-f0883fcb5fca"
-					(reference "D14")
+					(reference "D15")
 					(unit 1)
 				)
@@
 		(dnp no)
 		(fields_autoplaced yes)
-		(property "Reference" "R28"
+		(property "Reference" "R26"
 			(at 146.05 113.03 90)
 			(effects
@@
 			(project "Precision Clock"
 				(path "/c9a8ff63-a0d1-4125-9dd1-40fb53daf536/47769572-a111-4c65-a7b3-f0883fcb5fca"
-					(reference "R28")
+					(reference "R26")
 					(unit 1)
 				)
@@
 		(dnp no)
 		(fields_autoplaced yes)
-		(property "Reference" "C30"
+		(property "Reference" "C33"
 			(at 232.41 111.7599 0)
 			(effects
@@
 			(project "Precision Clock"
 				(path "/c9a8ff63-a0d1-4125-9dd1-40fb53daf536/47769572-a111-4c65-a7b3-f0883fcb5fca"
-					(reference "C30")
+					(reference "C33")
 					(unit 1)
 				)
@@
 		(dnp no)
 		(fields_autoplaced yes)
-		(property "Reference" "R31"
+		(property "Reference" "R28"
 			(at 138.43 57.1499 0)
 			(effects
@@
 			(project ""
 				(path "/c9a8ff63-a0d1-4125-9dd1-40fb53daf536/47769572-a111-4c65-a7b3-f0883fcb5fca"
-					(reference "R31")
+					(reference "R28")
 					(unit 1)
 				)
@@
 		(dnp no)
 		(fields_autoplaced yes)
-		(property "Reference" "R32"
+		(property "Reference" "R29"
 			(at 97.79 57.1499 0)
 			(effects
@@
 			(project "Precision Clock"
 				(path "/c9a8ff63-a0d1-4125-9dd1-40fb53daf536/47769572-a111-4c65-a7b3-f0883fcb5fca"
-					(reference "R32")
+					(reference "R29")
 					(unit 1)
 				)
@@
 		(on_board yes)
 		(dnp no)
-		(property "Reference" "D13"
+		(property "Reference" "D16"
 			(at 207.518 59.944 90)
 			(effects
@@
 			(project "Precision Clock"
 				(path "/c9a8ff63-a0d1-4125-9dd1-40fb53daf536/47769572-a111-4c65-a7b3-f0883fcb5fca"
-					(reference "D13")
-					(unit 1)
-				)
+					(reference "D16")
+					(unit 1)
+				)
