File: Temperature, Humidity & Pressure Sensor.kicad_sch (KiCad schematic)
At the start: 7 parts, among them U16 BME280

Commit message: In Production
Parts:
- U2: renamed from U16; LCSC (none) -> C92489
- renumbered C4 to C2, C2 to C3, R3 to R2, R2 to R3
Changed lines of the file:
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@@
 			)
 		)
-		(column_widths 20.32 48.26)
-		(row_heights 6.35 3.81 3.81 3.81 3.81 3.81 3.81)
+		(column_widths 20.32 24.13)
+		(row_heights 6.35 3.81 3.81 3.81)
 		(cells
 			(table_cell "Current Consumption "
 				(exclude_from_sim no)
-				(at 95.25 158.75 0)
+				(at 128.27 166.37 0)
 				(size 20.32 6.35)
 				(margins 0.9525 0.9525 0.9525 0.9525)
@@
 			(table_cell "Operation"
 				(exclude_from_sim no)
-				(at 115.57 158.75 0)
-				(size 48.26 6.35)
+				(at 148.59 166.37 0)
+				(size 24.13 6.35)
 				(margins 0.9525 0.9525 0.9525 0.9525)
 				(span 1 1)
@@
 				)
 			)
-			(table_cell "2.2uA"
+			(table_cell "1.8uA"
 				(exclude_from_sim no)
-				(at 95.25 165.1 0)
+				(at 128.27 172.72 0)
 				(size 20.32 3.81)
 				(margins 0.9525 0.9525 0.9525 0.9525)
@@
 			(table_cell "H/T @ 1Hz"
 				(exclude_from_sim no)
-				(at 115.57 165.1 0)
-				(size 48.26 3.81)
+				(at 148.59 172.72 0)
+				(size 24.13 3.81)
 				(margins 0.9525 0.9525 0.9525 0.9525)
 				(span 1 1)
@@
 				)
 			)
-			(table_cell "3.1uA "
+			(table_cell "2.8uA"
 				(exclude_from_sim no)
-				(at 95.25 168.91 0)
+				(at 128.27 176.53 0)
 				(size 20.32 3.81)
 				(margins 0.9525 0.9525 0.9525 0.9525)
@@
 			(table_cell "P/T @ 1Hz"
 				(exclude_from_sim no)
-				(at 115.57 168.91 0)
-				(size 48.26 3.81)
+				(at 148.59 176.53 0)
+				(size 24.13 3.81)
 				(margins 0.9525 0.9525 0.9525 0.9525)
 				(span 1 1)
@@
 				)
 			)
-			(table_cell "4.2uA "
+			(table_cell "3.6uA"
 				(exclude_from_sim no)
-				(at 95.25 172.72 0)
+				(at 128.27 180.34 0)
 				(size 20.32 3.81)
 				(margins 0.9525 0.9525 0.9525 0.9525)
@@
 			(table_cell "H/T/P @ 1Hz"
 				(exclude_from_sim no)
-				(at 115.57 172.72 0)
-				(size 48.26 3.81)
-				(margins 0.9525 0.9525 0.9525 0.9525)
-				(span 1 1)
-				(fill
-					(type none)
-				)
-				(effects
-					(font
-						(size 1.27 1.27)
-					)
-					(justify left top)
-				)
-			)
-			(table_cell "50uA"
-				(exclude_from_sim no)
-				(at 95.25 176.53 0)
-				(size 20.32 3.81)
-				(margins 0.9525 0.9525 0.9525 0.9525)
-				(span 1 1)
-				(fill
-					(type none)
-				)
-				(effects
-					(font
-						(size 1.27 1.27)
-					)
-					(justify left top)
-				)
-			)
-			(table_cell "H/T/P/AQI in Ultra low power mode"
-				(exclude_from_sim no)
-				(at 115.57 176.53 0)
-				(size 48.26 3.81)
-				(margins 0.9525 0.9525 0.9525 0.9525)
-				(span 1 1)
-				(fill
-					(type none)
-				)
-				(effects
-					(font
-						(size 1.27 1.27)
-					)
-					(justify left top)
-				)
-			)
-			(table_cell "500uA"
-				(exclude_from_sim no)
-				(at 95.25 180.34 0)
-				(size 20.32 3.81)
-				(margins 0.9525 0.9525 0.9525 0.9525)
-				(span 1 1)
-				(fill
-					(type none)
-				)
-				(effects
-					(font
-						(size 1.27 1.27)
-					)
-					(justify left top)
-				)
-			)
-			(table_cell "H/T/P/AQI in low power mode"
-				(exclude_from_sim no)
-				(at 115.57 180.34 0)
-				(size 48.26 3.81)
-				(margins 0.9525 0.9525 0.9525 0.9525)
-				(span 1 1)
-				(fill
-					(type none)
-				)
-				(effects
-					(font
-						(size 1.27 1.27)
-					)
-					(justify left top)
-				)
-			)
-			(table_cell "3.1mA"
-				(exclude_from_sim no)
-				(at 95.25 184.15 0)
-				(size 20.32 3.81)
-				(margins 0.9525 0.9525 0.9525 0.9525)
-				(span 1 1)
-				(fill
-					(type none)
-				)
-				(effects
-					(font
-						(size 1.27 1.27)
-					)
-					(justify left top)
-				)
-			)
-			(table_cell "Standard Gas scan mode"
-				(exclude_from_sim no)
-				(at 115.57 184.15 0)
-				(size 48.26 3.81)
+				(at 148.59 180.34 0)
+				(size 24.13 3.81)
 				(margins 0.9525 0.9525 0.9525 0.9525)
 				(span 1 1)
@@
 		(on_board yes)
 		(dnp no)
-		(fields_autoplaced yes)
-		(property "Reference" "U16"
-			(at 118.11 99.0599 0)
+		(property "Reference" "U2"
+			(at 117.856 97.536 0)
 			(effects
 				(font
@@
 		)
 		(property "Value" "BME280"
-			(at 118.11 101.5999 0)
+			(at 117.856 100.076 0)
 			(effects
 				(font
@@
 			)
 		)
+		(property "LCSC" "C92489"
+			(at 117.602 102.6161 0)
+			(effects
+				(font
+					(size 1.27 1.27)
+				)
+				(justify right)
+			)
+		)
 		(pin "6"
 		)
@@
 		)
 		(instances
-			(project ""
-				(path "/c9a8ff63-a0d1-4125-9dd1-40fb53daf536/cc882cab-fb20-4552-b867-43569dfc2d06"
-					(reference "U16")
+			(project "Precision Clock"
+				(path "/c9a8ff63-a0d1-4125-9dd1-40fb53daf536/cc882cab-fb20-4552-b867-43569dfc2d06"
+					(reference "U2")
 					(unit 1)
 				)
@@
 		)
 		(instances
-			(project ""
+			(project "Precision Clock"
 				(path "/c9a8ff63-a0d1-4125-9dd1-40fb53daf536/cc882cab-fb20-4552-b867-43569dfc2d06"
 					(reference "#PWR099")
@@
 		(dnp no)
 		(fields_autoplaced yes)
-		(property "Reference" "C4"
+		(property "Reference" "C2"
 			(at 92.71 88.8999 0)
 			(effects
@@
 			(project "Precision Clock"
 				(path "/c9a8ff63-a0d1-4125-9dd1-40fb53daf536/cc882cab-fb20-4552-b867-43569dfc2d06"
-					(reference "C4")
+					(reference "C2")
 					(unit 1)
 				)
@@
 		)
 		(instances
-			(project ""
+			(project "Precision Clock"
 				(path "/c9a8ff63-a0d1-4125-9dd1-40fb53daf536/cc882cab-fb20-4552-b867-43569dfc2d06"
 					(reference "TP2")
@@
 		(dnp no)
 		(fields_autoplaced yes)
-		(property "Reference" "R3"
+		(property "Reference" "R2"
 			(at 173.99 90.1699 0)
 			(effects
@@
 			(project "Precision Clock"
 				(path "/c9a8ff63-a0d1-4125-9dd1-40fb53daf536/cc882cab-fb20-4552-b867-43569dfc2d06"
-					(reference "R3")
+					(reference "R2")
 					(unit 1)
 				)
@@
 		)
 		(instances
-			(project ""
+			(project "Precision Clock"
 				(path "/c9a8ff63-a0d1-4125-9dd1-40fb53daf536/cc882cab-fb20-4552-b867-43569dfc2d06"
 					(reference "#PWR0102")
@@
 		(dnp no)
 		(fields_autoplaced yes)
-		(property "Reference" "C2"
+		(property "Reference" "C3"
 			(at 105.41 88.8999 0)
 			(effects
@@
 		)
 		(instances
-			(project ""
-				(path "/c9a8ff63-a0d1-4125-9dd1-40fb53daf536/cc882cab-fb20-4552-b867-43569dfc2d06"
-					(reference "C2")
+			(project "Precision Clock"
+				(path "/c9a8ff63-a0d1-4125-9dd1-40fb53daf536/cc882cab-fb20-4552-b867-43569dfc2d06"
+					(reference "C3")
 					(unit 1)
 				)
@@
 		(on_board yes)
 		(dnp no)
-		(fields_autoplaced yes)
 		(property "Reference" "#PWR098"
 			(at 88.9 104.14 0)
@@
 		(dnp no)
 		(fields_autoplaced yes)
-		(property "Reference" "R2"
+		(property "Reference" "R3"
 			(at 161.29 90.1699 0)
 			(effects
@@
 		)
 		(instances
-			(project ""
-				(path "/c9a8ff63-a0d1-4125-9dd1-40fb53daf536/cc882cab-fb20-4552-b867-43569dfc2d06"
-					(reference "R2")
+			(project "Precision Clock"
+				(path "/c9a8ff63-a0d1-4125-9dd1-40fb53daf536/cc882cab-fb20-4552-b867-43569dfc2d06"
+					(reference "R3")
 					(unit 1)
 				)
@@
 		)
 		(instances
-			(project ""
+			(project "Precision Clock"
 				(path "/c9a8ff63-a0d1-4125-9dd1-40fb53daf536/cc882cab-fb20-4552-b867-43569dfc2d06"
 					(reference "#PWR0101")
@@
 		)
 		(instances
-			(project ""
+			(project "Precision Clock"
 				(path "/c9a8ff63-a0d1-4125-9dd1-40fb53daf536/cc882cab-fb20-4552-b867-43569dfc2d06"
 					(reference "#PWR0100")
