File: power.kicad_sch (KiCad schematic)
At the start: 34 parts, among them Q1 DMN3008SFG, Q2 DMN3008SFG, U3 AP2127K-3.3, U4 AP33771C

Commit message: Major Changes
Parts:
- D10: renamed from D9; LCSC C364551 -> C364556
- D11: renamed from D10; LCSC C364551 -> C364556
- D12: renamed from D11; LCSC C364551 -> C364556
- D9: renamed from D8; LCSC C364551 -> C364556
- R10: renamed from R8; value 510R -> 750R
- R12: renamed from R10; value 510R -> 750R
- R15: renamed from R13; value 510R -> 750R
- R6: renamed from R4; value 510R -> 750R
- R9: renamed from R7; value 510R -> 750R
- renumbered R9 to R11, R11 to R13, R12 to R14, R3 to R5, R5 to R7, R6 to R8

Commit message: Verification
Parts:
- renumbered C17 to C10, C19 to C12, C25 to C13, C22 to C34, C26 to C35, C24 to C36, C18 to C38, C15 to C39, C16 to C41, C23 to C7, C20 to C8, C21 to C9, D9 to D1, D12 to D10, D10 to D11, D11 to D12, JP2 to JP1, JP1 to JP2, R11 to R10, R14 to R11, R8 to R13, R15 to R14, R12 to R17, R9 to R18, R13 to R33, R10 to R34, R7 to R5, R6 to R8, R5 to R9, U3 to U5, U4 to U9
Connections:
- net at Q1.1 (S), Q1.2 (S), Q1.3 (S): now also C8.1, C9.1, R13.2, U9.3 (VCC); no longer Q2.5 (D)
- new net: Q1.5 (D), Q2.5 (D)
Other:
- title: Power Regulation -> Power Negotiation & Regulation
- moved on the sheet: Q1

Commit message: Encoder placement
Parts:
- renumbered C13 to C10, C10 to C12, C7 to C13, C9 to C14, C36 to C35, C38 to C36, C35 to C37, C41 to C40, C39 to C41, C12 to C9, D12 to D11, D11 to D12, D1 to D2, D10 to D3, Q2 to Q1, Q1 to Q2, R13 to R11, R11 to R13, R10 to R14, R14 to R15, R18 to R17, R17 to R18, R9 to R5, R8 to R6, R5 to R8
Changed lines of the file:
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@@
 		(on_board yes)
 		(dnp no)
-		(property "Reference" "Q1"
+		(property "Reference" "Q2"
 			(at 209.55 23.622 90)
 			(effects
@@
 			(project ""
 				(path "/c9a8ff63-a0d1-4125-9dd1-40fb53daf536/8ce44042-2af7-42d8-9728-8ac0b976522a"
-					(reference "Q1")
+					(reference "Q2")
 					(unit 1)
 				)
@@
 		(dnp no)
 		(fields_autoplaced yes)
-		(property "Reference" "C12"
+		(property "Reference" "C9"
 			(at 156.21 36.8299 0)
 			(effects
@@
 			(project "Precision Clock"
 				(path "/c9a8ff63-a0d1-4125-9dd1-40fb53daf536/8ce44042-2af7-42d8-9728-8ac0b976522a"
-					(reference "C12")
+					(reference "C9")
 					(unit 1)
 				)
@@
 		(dnp no)
 		(fields_autoplaced yes)
-		(property "Reference" "C36"
+		(property "Reference" "C35"
 			(at 248.92 36.8299 0)
 			(effects
@@
 			(project "Precision Clock"
 				(path "/c9a8ff63-a0d1-4125-9dd1-40fb53daf536/8ce44042-2af7-42d8-9728-8ac0b976522a"
-					(reference "C36")
+					(reference "C35")
 					(unit 1)
 				)
@@
 		(dnp no)
 		(fields_autoplaced yes)
-		(property "Reference" "R5"
+		(property "Reference" "R8"
 			(at 146.05 83.8199 0)
 			(effects
@@
 			(project "Precision Clock"
 				(path "/c9a8ff63-a0d1-4125-9dd1-40fb53daf536/8ce44042-2af7-42d8-9728-8ac0b976522a"
-					(reference "R5")
+					(reference "R8")
 					(unit 1)
 				)
@@
 		(dnp no)
 		(fields_autoplaced yes)
-		(property "Reference" "R13"
+		(property "Reference" "R11"
 			(at 171.45 25.4 90)
 			(effects
@@
 			(project ""
 				(path "/c9a8ff63-a0d1-4125-9dd1-40fb53daf536/8ce44042-2af7-42d8-9728-8ac0b976522a"
-					(reference "R13")
+					(reference "R11")
 					(unit 1)
 				)
@@
 		(dnp no)
 		(fields_autoplaced yes)
-		(property "Reference" "C10"
+		(property "Reference" "C12"
 			(at 130.81 36.8299 0)
 			(effects
@@
 			(project ""
 				(path "/c9a8ff63-a0d1-4125-9dd1-40fb53daf536/8ce44042-2af7-42d8-9728-8ac0b976522a"
-					(reference "C10")
+					(reference "C12")
 					(unit 1)
 				)
@@
 		(on_board yes)
 		(dnp no)
-		(property "Reference" "D11"
+		(property "Reference" "D12"
 			(at 175.514 130.81 90)
 			(effects
@@
 			(project "Precision Clock"
 				(path "/c9a8ff63-a0d1-4125-9dd1-40fb53daf536/8ce44042-2af7-42d8-9728-8ac0b976522a"
-					(reference "D11")
+					(reference "D12")
 					(unit 1)
 				)
@@
 		(dnp no)
 		(fields_autoplaced yes)
-		(property "Reference" "R9"
+		(property "Reference" "R5"
 			(at 135.89 83.8199 0)
 			(effects
@@
 			(project ""
 				(path "/c9a8ff63-a0d1-4125-9dd1-40fb53daf536/8ce44042-2af7-42d8-9728-8ac0b976522a"
-					(reference "R9")
+					(reference "R5")
 					(unit 1)
 				)
@@
 		(dnp no)
 		(fields_autoplaced yes)
-		(property "Reference" "C39"
+		(property "Reference" "C41"
 			(at 35.56 43.1799 0)
 			(effects
@@
 			(project ""
 				(path "/c9a8ff63-a0d1-4125-9dd1-40fb53daf536/8ce44042-2af7-42d8-9728-8ac0b976522a"
-					(reference "C39")
+					(reference "C41")
 					(unit 1)
 				)
@@
 		(dnp no)
 		(fields_autoplaced yes)
-		(property "Reference" "R8"
+		(property "Reference" "R6"
 			(at 142.24 144.7799 0)
 			(effects
@@
 			(project ""
 				(path "/c9a8ff63-a0d1-4125-9dd1-40fb53daf536/8ce44042-2af7-42d8-9728-8ac0b976522a"
-					(reference "R8")
+					(reference "R6")
 					(unit 1)
 				)
@@
 		(dnp no)
 		(fields_autoplaced yes)
-		(property "Reference" "R11"
+		(property "Reference" "R13"
 			(at 237.49 83.8199 0)
 			(effects
@@
 			(project "Precision Clock"
 				(path "/c9a8ff63-a0d1-4125-9dd1-40fb53daf536/8ce44042-2af7-42d8-9728-8ac0b976522a"
-					(reference "R11")
+					(reference "R13")
 					(unit 1)
 				)
@@
 		(on_board yes)
 		(dnp no)
-		(property "Reference" "D1"
+		(property "Reference" "D2"
 			(at 143.764 130.81 90)
 			(effects
@@
 			(project ""
 				(path "/c9a8ff63-a0d1-4125-9dd1-40fb53daf536/8ce44042-2af7-42d8-9728-8ac0b976522a"
-					(reference "D1")
+					(reference "D2")
 					(unit 1)
 				)
@@
 		(dnp no)
 		(fields_autoplaced yes)
-		(property "Reference" "C13"
+		(property "Reference" "C10"
 			(at 251.46 83.8199 0)
 			(effects
@@
 			(project "Precision Clock"
 				(path "/c9a8ff63-a0d1-4125-9dd1-40fb53daf536/8ce44042-2af7-42d8-9728-8ac0b976522a"
-					(reference "C13")
+					(reference "C10")
 					(unit 1)
 				)
@@
 		(dnp no)
 		(fields_autoplaced yes)
-		(property "Reference" "C7"
+		(property "Reference" "C13"
 			(at 226.06 85.0899 0)
 			(effects
@@
 			(project "Precision Clock"
 				(path "/c9a8ff63-a0d1-4125-9dd1-40fb53daf536/8ce44042-2af7-42d8-9728-8ac0b976522a"
-					(reference "C7")
+					(reference "C13")
 					(unit 1)
 				)
@@
 		(dnp no)
 		(fields_autoplaced yes)
-		(property "Reference" "C38"
+		(property "Reference" "C36"
 			(at 143.51 36.8299 0)
 			(effects
@@
 			(project "Precision Clock"
 				(path "/c9a8ff63-a0d1-4125-9dd1-40fb53daf536/8ce44042-2af7-42d8-9728-8ac0b976522a"
-					(reference "C38")
+					(reference "C36")
 					(unit 1)
 				)
@@
 		(dnp no)
 		(fields_autoplaced yes)
-		(property "Reference" "C9"
+		(property "Reference" "C14"
 			(at 200.66 36.8299 0)
 			(effects
@@
 			(project "Precision Clock"
 				(path "/c9a8ff63-a0d1-4125-9dd1-40fb53daf536/8ce44042-2af7-42d8-9728-8ac0b976522a"
-					(reference "C9")
+					(reference "C14")
 					(unit 1)
 				)
@@
 		(dnp no)
 		(fields_autoplaced yes)
-		(property "Reference" "R14"
+		(property "Reference" "R15"
 			(at 243.84 146.0499 0)
 			(effects
@@
 			(project "Precision Clock"
 				(path "/c9a8ff63-a0d1-4125-9dd1-40fb53daf536/8ce44042-2af7-42d8-9728-8ac0b976522a"
-					(reference "R14")
+					(reference "R15")
 					(unit 1)
 				)
@@
 		(on_board yes)
 		(dnp no)
-		(property "Reference" "Q2"
+		(property "Reference" "Q1"
 			(at 224.79 23.622 90)
 			(effects
@@
 			(project "Precision Clock"
 				(path "/c9a8ff63-a0d1-4125-9dd1-40fb53daf536/8ce44042-2af7-42d8-9728-8ac0b976522a"
-					(reference "Q2")
+					(reference "Q1")
 					(unit 1)
 				)
@@
 		(dnp no)
 		(fields_autoplaced yes)
-		(property "Reference" "C41"
+		(property "Reference" "C40"
 			(at 73.66 43.1799 0)
 			(effects
@@
 			(project "Precision Clock"
 				(path "/c9a8ff63-a0d1-4125-9dd1-40fb53daf536/8ce44042-2af7-42d8-9728-8ac0b976522a"
-					(reference "C41")
+					(reference "C40")
 					(unit 1)
 				)
@@
 		(dnp no)
 		(fields_autoplaced yes)
-		(property "Reference" "R10"
+		(property "Reference" "R14"
 			(at 212.09 85.0899 0)
 			(effects
@@
 			(project ""
 				(path "/c9a8ff63-a0d1-4125-9dd1-40fb53daf536/8ce44042-2af7-42d8-9728-8ac0b976522a"
-					(reference "R10")
+					(reference "R14")
 					(unit 1)
 				)
@@
 		(dnp no)
 		(fields_autoplaced yes)
-		(property "Reference" "C35"
+		(property "Reference" "C37"
 			(at 261.62 36.8299 0)
 			(effects
@@
 			(project "Precision Clock"
 				(path "/c9a8ff63-a0d1-4125-9dd1-40fb53daf536/8ce44042-2af7-42d8-9728-8ac0b976522a"
-					(reference "C35")
+					(reference "C37")
 					(unit 1)
 				)
@@
 		(dnp no)
 		(fields_autoplaced yes)
-		(property "Reference" "R17"
+		(property "Reference" "R18"
 			(at 218.44 144.7799 0)
 			(effects
@@
 			(project "Precision Clock"
 				(path "/c9a8ff63-a0d1-4125-9dd1-40fb53daf536/8ce44042-2af7-42d8-9728-8ac0b976522a"
-					(reference "R17")
+					(reference "R18")
 					(unit 1)
 				)
@@
 		(dnp no)
 		(fields_autoplaced yes)
-		(property "Reference" "R18"
+		(property "Reference" "R17"
 			(at 173.99 144.7799 0)
 			(effects
@@
 			(project "Precision Clock"
 				(path "/c9a8ff63-a0d1-4125-9dd1-40fb53daf536/8ce44042-2af7-42d8-9728-8ac0b976522a"
-					(reference "R18")
+					(reference "R17")
 					(unit 1)
 				)
@@
 		(on_board yes)
 		(dnp no)
-		(property "Reference" "D10"
+		(property "Reference" "D3"
 			(at 245.364 132.08 90)
 			(effects
@@
 			(project "Precision Clock"
 				(path "/c9a8ff63-a0d1-4125-9dd1-40fb53daf536/8ce44042-2af7-42d8-9728-8ac0b976522a"
-					(reference "D10")
+					(reference "D3")
 					(unit 1)
 				)
@@
 		(on_board yes)
 		(dnp no)
-		(property "Reference" "D12"
+		(property "Reference" "D11"
 			(at 207.264 130.81 90)
 			(effects
@@
 			(project "Precision Clock"
 				(path "/c9a8ff63-a0d1-4125-9dd1-40fb53daf536/8ce44042-2af7-42d8-9728-8ac0b976522a"
-					(reference "D12")
+					(reference "D11")
 					(unit 1)
 				)

Commit message: Minor changes
Parts:
- renumbered C13 to C10, C8 to C12, C34 to C33, C36 to C34, C40 to C38, C41 to C40, C9 to C7, C10 to C8, C12 to C9, D2 to D1, D12 to D11, D11 to D12, D3 to D6, JP2 to JP1, JP1 to JP2, R5 to R13, R6 to R14, R8 to R15, R13 to R16, R14 to R17, R11 to R18, R15 to R22, R18 to R23, R17 to R24, R33 to R31, R34 to R32, U5 to U4
Changed lines of the file:
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@@
 		(dnp no)
 		(fields_autoplaced yes)
-		(property "Reference" "C34"
+		(property "Reference" "C33"
 			(at 200.66 87.6299 0)
 			(effects
@@
 			(project ""
 				(path "/c9a8ff63-a0d1-4125-9dd1-40fb53daf536/8ce44042-2af7-42d8-9728-8ac0b976522a"
-					(reference "C34")
+					(reference "C33")
 					(unit 1)
 				)
@@
 		(dnp no)
 		(fields_autoplaced yes)
-		(property "Reference" "C9"
+		(property "Reference" "C7"
 			(at 156.21 36.8299 0)
 			(effects
@@
 			(project "Precision Clock"
 				(path "/c9a8ff63-a0d1-4125-9dd1-40fb53daf536/8ce44042-2af7-42d8-9728-8ac0b976522a"
-					(reference "C9")
+					(reference "C7")
 					(unit 1)
 				)
@@
 		(on_board yes)
 		(dnp no)
-		(property "Reference" "U5"
+		(property "Reference" "U4"
 			(at 50.8 29.464 0)
 			(effects
@@
 			(project ""
 				(path "/c9a8ff63-a0d1-4125-9dd1-40fb53daf536/8ce44042-2af7-42d8-9728-8ac0b976522a"
-					(reference "U5")
+					(reference "U4")
 					(unit 1)
 				)
@@
 		(dnp no)
 		(fields_autoplaced yes)
-		(property "Reference" "JP2"
+		(property "Reference" "JP1"
 			(at 50.8 120.65 0)
 			(effects
@@
 			(project ""
 				(path "/c9a8ff63-a0d1-4125-9dd1-40fb53daf536/8ce44042-2af7-42d8-9728-8ac0b976522a"
-					(reference "JP2")
+					(reference "JP1")
 					(unit 1)
 				)
@@
 		(dnp no)
 		(fields_autoplaced yes)
-		(property "Reference" "R8"
+		(property "Reference" "R15"
 			(at 146.05 83.8199 0)
 			(effects
@@
 			(project "Precision Clock"
 				(path "/c9a8ff63-a0d1-4125-9dd1-40fb53daf536/8ce44042-2af7-42d8-9728-8ac0b976522a"
-					(reference "R8")
+					(reference "R15")
 					(unit 1)
 				)
@@
 		(dnp no)
 		(fields_autoplaced yes)
-		(property "Reference" "R11"
+		(property "Reference" "R18"
 			(at 171.45 25.4 90)
 			(effects
@@
 			(project ""
 				(path "/c9a8ff63-a0d1-4125-9dd1-40fb53daf536/8ce44042-2af7-42d8-9728-8ac0b976522a"
-					(reference "R11")
+					(reference "R18")
 					(unit 1)
 				)
@@
 		(dnp no)
 		(fields_autoplaced yes)
-		(property "Reference" "C12"
+		(property "Reference" "C9"
 			(at 130.81 36.8299 0)
 			(effects
@@
 			(project ""
 				(path "/c9a8ff63-a0d1-4125-9dd1-40fb53daf536/8ce44042-2af7-42d8-9728-8ac0b976522a"
-					(reference "C12")
+					(reference "C9")
 					(unit 1)
 				)
@@
 		(on_board yes)
 		(dnp no)
-		(property "Reference" "D12"
+		(property "Reference" "D11"
 			(at 175.514 130.81 90)
 			(effects
@@
 			(project "Precision Clock"
 				(path "/c9a8ff63-a0d1-4125-9dd1-40fb53daf536/8ce44042-2af7-42d8-9728-8ac0b976522a"
-					(reference "D12")
+					(reference "D11")
 					(unit 1)
 				)
@@
 		(dnp no)
 		(fields_autoplaced yes)
-		(property "Reference" "R5"
+		(property "Reference" "R13"
 			(at 135.89 83.8199 0)
 			(effects
@@
 			(project ""
 				(path "/c9a8ff63-a0d1-4125-9dd1-40fb53daf536/8ce44042-2af7-42d8-9728-8ac0b976522a"
-					(reference "R5")
+					(reference "R13")
 					(unit 1)
 				)
@@
 		(dnp no)
 		(fields_autoplaced yes)
-		(property "Reference" "C41"
+		(property "Reference" "C40"
 			(at 35.56 43.1799 0)
 			(effects
@@
 			(project ""
 				(path "/c9a8ff63-a0d1-4125-9dd1-40fb53daf536/8ce44042-2af7-42d8-9728-8ac0b976522a"
-					(reference "C41")
+					(reference "C40")
 					(unit 1)
 				)
@@
 		(dnp no)
 		(fields_autoplaced yes)
-		(property "Reference" "R6"
+		(property "Reference" "R14"
 			(at 142.24 144.7799 0)
 			(effects
@@
 			(project ""
 				(path "/c9a8ff63-a0d1-4125-9dd1-40fb53daf536/8ce44042-2af7-42d8-9728-8ac0b976522a"
-					(reference "R6")
+					(reference "R14")
 					(unit 1)
 				)
@@
 		(dnp no)
 		(fields_autoplaced yes)
-		(property "Reference" "R13"
+		(property "Reference" "R16"
 			(at 237.49 83.8199 0)
 			(effects
@@
 			(project "Precision Clock"
 				(path "/c9a8ff63-a0d1-4125-9dd1-40fb53daf536/8ce44042-2af7-42d8-9728-8ac0b976522a"
-					(reference "R13")
+					(reference "R16")
 					(unit 1)
 				)
@@
 		(on_board yes)
 		(dnp no)
-		(property "Reference" "D2"
+		(property "Reference" "D1"
 			(at 143.764 130.81 90)
 			(effects
@@
 			(project ""
 				(path "/c9a8ff63-a0d1-4125-9dd1-40fb53daf536/8ce44042-2af7-42d8-9728-8ac0b976522a"
-					(reference "D2")
+					(reference "D1")
 					(unit 1)
 				)
@@
 		(dnp no)
 		(fields_autoplaced yes)
-		(property "Reference" "C10"
+		(property "Reference" "C8"
 			(at 251.46 83.8199 0)
 			(effects
@@
 			(project "Precision Clock"
 				(path "/c9a8ff63-a0d1-4125-9dd1-40fb53daf536/8ce44042-2af7-42d8-9728-8ac0b976522a"
-					(reference "C10")
+					(reference "C8")
 					(unit 1)
 				)
@@
 		(dnp no)
 		(fields_autoplaced yes)
-		(property "Reference" "C13"
+		(property "Reference" "C10"
 			(at 226.06 85.0899 0)
 			(effects
@@
 			(project "Precision Clock"
 				(path "/c9a8ff63-a0d1-4125-9dd1-40fb53daf536/8ce44042-2af7-42d8-9728-8ac0b976522a"
-					(reference "C13")
+					(reference "C10")
 					(unit 1)
 				)
@@
 		(dnp no)
 		(fields_autoplaced yes)
-		(property "Reference" "C36"
+		(property "Reference" "C34"
 			(at 143.51 36.8299 0)
 			(effects
@@
 			(project "Precision Clock"
 				(path "/c9a8ff63-a0d1-4125-9dd1-40fb53daf536/8ce44042-2af7-42d8-9728-8ac0b976522a"
-					(reference "C36")
+					(reference "C34")
 					(unit 1)
 				)
@@
 		(dnp no)
 		(fields_autoplaced yes)
-		(property "Reference" "R33"
+		(property "Reference" "R31"
 			(at 219.71 46.9899 0)
 			(effects
@@
 			(project ""
 				(path "/c9a8ff63-a0d1-4125-9dd1-40fb53daf536/8ce44042-2af7-42d8-9728-8ac0b976522a"
-					(reference "R33")
+					(reference "R31")
 					(unit 1)
 				)
@@
 		(dnp no)
 		(fields_autoplaced yes)
-		(property "Reference" "R15"
+		(property "Reference" "R22"
 			(at 243.84 146.0499 0)
 			(effects
@@
 			(project "Precision Clock"
 				(path "/c9a8ff63-a0d1-4125-9dd1-40fb53daf536/8ce44042-2af7-42d8-9728-8ac0b976522a"
-					(reference "R15")
+					(reference "R22")
 					(unit 1)
 				)
@@
 		(dnp no)
 		(fields_autoplaced yes)
-		(property "Reference" "R34"
+		(property "Reference" "R32"
 			(at 205.74 144.7799 0)
 			(effects
@@
 			(project "Precision Clock"
 				(path "/c9a8ff63-a0d1-4125-9dd1-40fb53daf536/8ce44042-2af7-42d8-9728-8ac0b976522a"
-					(reference "R34")
+					(reference "R32")
 					(unit 1)
 				)
@@
 		(dnp no)
 		(fields_autoplaced yes)
-		(property "Reference" "C40"
+		(property "Reference" "C38"
 			(at 73.66 43.1799 0)
 			(effects
@@
 			(project "Precision Clock"
 				(path "/c9a8ff63-a0d1-4125-9dd1-40fb53daf536/8ce44042-2af7-42d8-9728-8ac0b976522a"
-					(reference "C40")
+					(reference "C38")
 					(unit 1)
 				)
@@
 		(dnp no)
 		(fields_autoplaced yes)
-		(property "Reference" "C8"
+		(property "Reference" "C12"
 			(at 187.96 36.8299 0)
 			(effects
@@
 			(project "Precision Clock"
 				(path "/c9a8ff63-a0d1-4125-9dd1-40fb53daf536/8ce44042-2af7-42d8-9728-8ac0b976522a"
-					(reference "C8")
+					(reference "C12")
 					(unit 1)
 				)
@@
 		(dnp no)
 		(fields_autoplaced yes)
-		(property "Reference" "R14"
+		(property "Reference" "R17"
 			(at 212.09 85.0899 0)
 			(effects
@@
 			(project ""
 				(path "/c9a8ff63-a0d1-4125-9dd1-40fb53daf536/8ce44042-2af7-42d8-9728-8ac0b976522a"
-					(reference "R14")
+					(reference "R17")
 					(unit 1)
 				)
@@
 		(dnp no)
 		(fields_autoplaced yes)
-		(property "Reference" "R18"
+		(property "Reference" "R23"
 			(at 218.44 144.7799 0)
 			(effects
@@
 			(project "Precision Clock"
 				(path "/c9a8ff63-a0d1-4125-9dd1-40fb53daf536/8ce44042-2af7-42d8-9728-8ac0b976522a"
-					(reference "R18")
+					(reference "R23")
 					(unit 1)
 				)
@@
 		(dnp no)
 		(fields_autoplaced yes)
-		(property "Reference" "R17"
+		(property "Reference" "R24"
 			(at 173.99 144.7799 0)
 			(effects
@@
 			(project "Precision Clock"
 				(path "/c9a8ff63-a0d1-4125-9dd1-40fb53daf536/8ce44042-2af7-42d8-9728-8ac0b976522a"
-					(reference "R17")
+					(reference "R24")
 					(unit 1)
 				)
@@
 		(on_board yes)
 		(dnp no)
-		(property "Reference" "D3"
+		(property "Reference" "D6"
 			(at 245.364 132.08 90)
 			(effects
@@
 			(project "Precision Clock"
 				(path "/c9a8ff63-a0d1-4125-9dd1-40fb53daf536/8ce44042-2af7-42d8-9728-8ac0b976522a"
-					(reference "D3")
+					(reference "D6")
 					(unit 1)
 				)
@@
 		(dnp no)
 		(fields_autoplaced yes)
-		(property "Reference" "JP1"
+		(property "Reference" "JP2"
 			(at 50.8 139.7 0)
 			(effects
@@
 			(project "Precision Clock"
 				(path "/c9a8ff63-a0d1-4125-9dd1-40fb53daf536/8ce44042-2af7-42d8-9728-8ac0b976522a"
-					(reference "JP1")
+					(reference "JP2")
 					(unit 1)
 				)
@@
 		(on_board yes)
 		(dnp no)
-		(property "Reference" "D11"
+		(property "Reference" "D12"
 			(at 207.264 130.81 90)
 			(effects
@@
 			(project "Precision Clock"
 				(path "/c9a8ff63-a0d1-4125-9dd1-40fb53daf536/8ce44042-2af7-42d8-9728-8ac0b976522a"
-					(reference "D11")
+					(reference "D12")
 					(unit 1)
 				)

Commit message: Production files preparation
Parts:
- C10: renamed from C8; LCSC (none) -> C15195
- C11: renamed from C14; LCSC (none) -> C86275
- C12: LCSC (none) -> C86275
- C35: renamed from C33; LCSC (none) -> C29266
- C36: renamed from C35; LCSC (none) -> C1525
- C38: renamed from C37; LCSC (none) -> C86275
- C39: renamed from C34; LCSC (none) -> C1525
- C40: LCSC (none) -> C29266
- C41: renamed from C38; LCSC (none) -> C29266
- C6: renamed from C10; LCSC (none) -> C15195
- C7: renamed from C9; LCSC (none) -> C86275
- C9: renamed from C7; LCSC (none) -> C1525
- R11: renamed from R13; LCSC (none) -> C105872
- R12: renamed from R14; LCSC (none) -> C137936
- R14: renamed from R15; LCSC (none) -> C105872
- R16: LCSC (none) -> C60491
- R17: renamed from R22; LCSC (none) -> C137936
- R19: renamed from R18; LCSC (none) -> C92742
- R20: renamed from R17; LCSC (none) -> C137995
- R22: renamed from R23; LCSC (none) -> C137936
- R23: renamed from R24; LCSC (none) -> C137936
- R38: renamed from R31; LCSC (none) -> C105872
- R39: renamed from R32; LCSC (none) -> C137936
- U9: LCSC (none) -> C24735840
- renumbered D11 to D10, D12 to D11, D6 to D9, U4 to U5
