File: power.kicad_sch (KiCad schematic)
At the start: 34 parts, among them Q1 DMN3008SFG, Q2 DMN3008SFG, U5 AP2127K-3.3, U9 AP33771C

Commit message: In Production
Parts:
- renumbered C10 to C11, C11 to C12, C12 to C13, C6 to C14, C35 to C36, C36 to C37, C39 to C38, C38 to C39, C40 to C41, C41 to C42, D10 to D11, D11 to D12, D9 to D8, JP2 to JP1, JP1 to JP2, R14 to R11, R11 to R13, R20 to R17, R19 to R18, R17 to R19, R16 to R20
Changed lines of the file:
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@@
 		(dnp no)
 		(fields_autoplaced yes)
-		(property "Reference" "C35"
+		(property "Reference" "C36"
 			(at 200.66 87.6299 0)
 			(effects
@@
 			(project ""
 				(path "/c9a8ff63-a0d1-4125-9dd1-40fb53daf536/8ce44042-2af7-42d8-9728-8ac0b976522a"
-					(reference "C35")
+					(reference "C36")
 					(unit 1)
 				)
@@
 		(dnp no)
 		(fields_autoplaced yes)
-		(property "Reference" "JP1"
+		(property "Reference" "JP2"
 			(at 50.8 120.65 0)
 			(effects
@@
 			(project ""
 				(path "/c9a8ff63-a0d1-4125-9dd1-40fb53daf536/8ce44042-2af7-42d8-9728-8ac0b976522a"
-					(reference "JP1")
+					(reference "JP2")
 					(unit 1)
 				)
@@
 		(dnp no)
 		(fields_autoplaced yes)
-		(property "Reference" "C36"
+		(property "Reference" "C37"
 			(at 248.92 36.8299 0)
 			(effects
@@
 			(project "Precision Clock"
 				(path "/c9a8ff63-a0d1-4125-9dd1-40fb53daf536/8ce44042-2af7-42d8-9728-8ac0b976522a"
-					(reference "C36")
+					(reference "C37")
 					(unit 1)
 				)
@@
 		(dnp no)
 		(fields_autoplaced yes)
-		(property "Reference" "R14"
+		(property "Reference" "R11"
 			(at 146.05 83.8199 0)
 			(effects
@@
 			(project "Precision Clock"
 				(path "/c9a8ff63-a0d1-4125-9dd1-40fb53daf536/8ce44042-2af7-42d8-9728-8ac0b976522a"
-					(reference "R14")
+					(reference "R11")
 					(unit 1)
 				)
@@
 		(dnp no)
 		(fields_autoplaced yes)
-		(property "Reference" "R19"
+		(property "Reference" "R18"
 			(at 171.45 25.4 90)
 			(effects
@@
 			(project ""
 				(path "/c9a8ff63-a0d1-4125-9dd1-40fb53daf536/8ce44042-2af7-42d8-9728-8ac0b976522a"
-					(reference "R19")
+					(reference "R18")
 					(unit 1)
 				)
@@
 		(on_board yes)
 		(dnp no)
-		(property "Reference" "D10"
+		(property "Reference" "D11"
 			(at 175.514 130.81 90)
 			(effects
@@
 			(project "Precision Clock"
 				(path "/c9a8ff63-a0d1-4125-9dd1-40fb53daf536/8ce44042-2af7-42d8-9728-8ac0b976522a"
-					(reference "D10")
+					(reference "D11")
 					(unit 1)
 				)
@@
 		(dnp no)
 		(fields_autoplaced yes)
-		(property "Reference" "R11"
+		(property "Reference" "R13"
 			(at 135.89 83.8199 0)
 			(effects
@@
 			(project ""
 				(path "/c9a8ff63-a0d1-4125-9dd1-40fb53daf536/8ce44042-2af7-42d8-9728-8ac0b976522a"
-					(reference "R11")
+					(reference "R13")
 					(unit 1)
 				)
@@
 		(dnp no)
 		(fields_autoplaced yes)
-		(property "Reference" "C40"
+		(property "Reference" "C41"
 			(at 35.56 43.1799 0)
 			(effects
@@
 			(project ""
 				(path "/c9a8ff63-a0d1-4125-9dd1-40fb53daf536/8ce44042-2af7-42d8-9728-8ac0b976522a"
-					(reference "C40")
+					(reference "C41")
 					(unit 1)
 				)
@@
 		(dnp no)
 		(fields_autoplaced yes)
-		(property "Reference" "R16"
+		(property "Reference" "R20"
 			(at 237.49 83.8199 0)
 			(effects
@@
 			(project "Precision Clock"
 				(path "/c9a8ff63-a0d1-4125-9dd1-40fb53daf536/8ce44042-2af7-42d8-9728-8ac0b976522a"
-					(reference "R16")
+					(reference "R20")
 					(unit 1)
 				)
@@
 		(dnp no)
 		(fields_autoplaced yes)
-		(property "Reference" "C10"
+		(property "Reference" "C11"
 			(at 251.46 83.8199 0)
 			(effects
@@
 			(project "Precision Clock"
 				(path "/c9a8ff63-a0d1-4125-9dd1-40fb53daf536/8ce44042-2af7-42d8-9728-8ac0b976522a"
-					(reference "C10")
+					(reference "C11")
 					(unit 1)
 				)
@@
 		(dnp no)
 		(fields_autoplaced yes)
-		(property "Reference" "C6"
+		(property "Reference" "C14"
 			(at 226.06 85.0899 0)
 			(effects
@@
 			(project "Precision Clock"
 				(path "/c9a8ff63-a0d1-4125-9dd1-40fb53daf536/8ce44042-2af7-42d8-9728-8ac0b976522a"
-					(reference "C6")
+					(reference "C14")
 					(unit 1)
 				)
@@
 		(dnp no)
 		(fields_autoplaced yes)
-		(property "Reference" "C39"
+		(property "Reference" "C38"
 			(at 143.51 36.8299 0)
 			(effects
@@
 			(project "Precision Clock"
 				(path "/c9a8ff63-a0d1-4125-9dd1-40fb53daf536/8ce44042-2af7-42d8-9728-8ac0b976522a"
-					(reference "C39")
+					(reference "C38")
 					(unit 1)
 				)
@@
 		(dnp no)
 		(fields_autoplaced yes)
-		(property "Reference" "C11"
+		(property "Reference" "C12"
 			(at 200.66 36.8299 0)
 			(effects
@@
 			(project "Precision Clock"
 				(path "/c9a8ff63-a0d1-4125-9dd1-40fb53daf536/8ce44042-2af7-42d8-9728-8ac0b976522a"
-					(reference "C11")
+					(reference "C12")
 					(unit 1)
 				)
@@
 		(dnp no)
 		(fields_autoplaced yes)
-		(property "Reference" "R17"
+		(property "Reference" "R19"
 			(at 243.84 146.0499 0)
 			(effects
@@
 			(project "Precision Clock"
 				(path "/c9a8ff63-a0d1-4125-9dd1-40fb53daf536/8ce44042-2af7-42d8-9728-8ac0b976522a"
-					(reference "R17")
+					(reference "R19")
 					(unit 1)
 				)
@@
 		(dnp no)
 		(fields_autoplaced yes)
-		(property "Reference" "C41"
+		(property "Reference" "C42"
 			(at 73.66 43.1799 0)
 			(effects
@@
 			(project "Precision Clock"
 				(path "/c9a8ff63-a0d1-4125-9dd1-40fb53daf536/8ce44042-2af7-42d8-9728-8ac0b976522a"
-					(reference "C41")
+					(reference "C42")
 					(unit 1)
 				)
@@
 		(dnp no)
 		(fields_autoplaced yes)
-		(property "Reference" "C12"
+		(property "Reference" "C13"
 			(at 187.96 36.8299 0)
 			(effects
@@
 			(project "Precision Clock"
 				(path "/c9a8ff63-a0d1-4125-9dd1-40fb53daf536/8ce44042-2af7-42d8-9728-8ac0b976522a"
-					(reference "C12")
+					(reference "C13")
 					(unit 1)
 				)
@@
 		(dnp no)
 		(fields_autoplaced yes)
-		(property "Reference" "R20"
+		(property "Reference" "R17"
 			(at 212.09 85.0899 0)
 			(effects
@@
 			(project ""
 				(path "/c9a8ff63-a0d1-4125-9dd1-40fb53daf536/8ce44042-2af7-42d8-9728-8ac0b976522a"
-					(reference "R20")
+					(reference "R17")
 					(unit 1)
 				)
@@
 		(dnp no)
 		(fields_autoplaced yes)
-		(property "Reference" "C38"
+		(property "Reference" "C39"
 			(at 261.62 36.8299 0)
 			(effects
@@
 			(project "Precision Clock"
 				(path "/c9a8ff63-a0d1-4125-9dd1-40fb53daf536/8ce44042-2af7-42d8-9728-8ac0b976522a"
-					(reference "C38")
+					(reference "C39")
 					(unit 1)
 				)
@@
 		(on_board yes)
 		(dnp no)
-		(property "Reference" "D9"
+		(property "Reference" "D8"
 			(at 245.364 132.08 90)
 			(effects
@@
 			(project "Precision Clock"
 				(path "/c9a8ff63-a0d1-4125-9dd1-40fb53daf536/8ce44042-2af7-42d8-9728-8ac0b976522a"
-					(reference "D9")
+					(reference "D8")
 					(unit 1)
 				)
@@
 		(dnp no)
 		(fields_autoplaced yes)
-		(property "Reference" "JP2"
+		(property "Reference" "JP1"
 			(at 50.8 139.7 0)
 			(effects
@@
 			(project "Precision Clock"
 				(path "/c9a8ff63-a0d1-4125-9dd1-40fb53daf536/8ce44042-2af7-42d8-9728-8ac0b976522a"
-					(reference "JP2")
+					(reference "JP1")
 					(unit 1)
 				)
@@
 		(on_board yes)
 		(dnp no)
-		(property "Reference" "D11"
+		(property "Reference" "D12"
 			(at 207.264 130.81 90)
 			(effects
@@
 			(project "Precision Clock"
 				(path "/c9a8ff63-a0d1-4125-9dd1-40fb53daf536/8ce44042-2af7-42d8-9728-8ac0b976522a"
-					(reference "D11")
+					(reference "D12")
 					(unit 1)
 				)

Commit message: Push Button Replacement
Parts:
- removed D1: LED, precision_clock:LED_LiteON_LTST-C281KGKT, symbol Device:LED
- removed R12: 750R, Resistor_SMD:R_0402_1005Metric, symbol Device:R
- renumbered C7 to C10, C9 to C11, C37 to C13, C14 to C35, C41 to C37, C11 to C38, C38 to C39, C39 to C40, C36 to C6, C13 to C7, D12 to D11, D8 to D2, D11 to D4, JP2 to JP1, JP1 to JP2, Q2 to Q1, Q1 to Q2, R13 to R12, R11 to R14, R19 to R15, R18 to R17, R23 to R18, R39 to R19, R17 to R36, R20 to R37, U5 to U4
Other:
- note removed: "USB PWR OK"
- moved on the sheet: D11, D2, D4, R15, R18, R19, R22
