File: mcu.kicad_sch (KiCad schematic)
At the start: 34 parts, among them J2 USB_C_Receptacle, J3 Conn_ST_STDC14, SW2 B3U-1000P, SW3 B3U-1000P, U3 W25Q32JVZP, U4 STM32G0B0CET6, Y1 ECS-TXO-2520MV, Y2 Q13MC14620002

Commit message: Production Ready v2
Parts:
- U4: LCSC (none) -> C2826978
Changed lines of the file:
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@@
+			)
+		)
+		(property "LCSC" "C2826978"
+			(at 82.55 91.44 0)
+			(effects
+				(font
+					(size 1.27 1.27)
+				)
+				(hide yes)
 			)
 		)
