File: Precision Clock-backups/Precision Clock-2026-03-12_203712/Clock Display.kicad_sch (KiCad schematic)
At the start: 21 parts, among them U10 SA15-11SURKWA, U11 SA15-11SURKWA, U12 SA15-11SURKWA, U13 SA15-11SURKWA, U14 SA15-11SURKWA, U15 SA15-11SURKWA, U6 TLC5926, U7 TLC5926, U8 TLC5926

Commit message: Routing
Parts:
- added TP10: SCL, TestPoint:TestPoint_Pad_D1.0mm, symbol Connector:TestPoint
- added TP4: OE, TestPoint:TestPoint_Pad_D1.0mm, symbol Connector:TestPoint
- added TP5: SDI, TestPoint:TestPoint_Pad_D1.0mm, symbol Connector:TestPoint
- added TP7: LE, TestPoint:TestPoint_Pad_D1.0mm, symbol Connector:TestPoint
- added TP9: SDO, TestPoint:TestPoint_Pad_D1.0mm, symbol Connector:TestPoint
- renumbered C21 to C25, C23 to C26, C22 to C27, C35 to C36, C37 to C41, C39 to C43, C40 to C44, C41 to C45, C42 to C46, R25 to R23, R26 to R24, R27 to R25
Connections:
- net LE: now also TP7.1
- net OE: now also TP4.1
- net SCL: now also TP10.1
- net SDI: now also TP5.1
- net SDO: now also TP9.1
Other:
- note added: "Test Points"
