File: Precision Clock-backups/Precision Clock-2026-03-12_203712/MCU.kicad_sch (KiCad schematic)
At the start: 36 parts, among them J2 USB_C_Receptacle, J3 Conn_ST_STDC14, SW2 B3U-1000P, SW3 B3U-1000P, U3 W25Q32JVZP, U4 STM32G0B0CETx, Y1 Q13MC14620002, Y2 ECS-TXO-2520MV

Commit message: Routing
Parts:
- removed D18: LED, precision_clock:LED_LiteON_LTST-C281KGKT, symbol Device:LED
- removed R42, R43: 750R, Resistor_SMD:R_0402_1005Metric, symbol Device:R
- renumbered C15 to C16, C20 to C17, C17 to C18, C18 to C19, C16 to C20, C19 to C21, C14 to C24, C9 to C8, D2 to D1, D11 to D10, D6 to D5, D9 to D6, D5 to D7, D7 to D8, D8 to D9, R17 to R16, R22 to R20, R23 to R21, R5 to R4, R19 to R40, R24 to R41, R4 to R42, U3 to U16, U4 to U5
Connections:
- net ENC_A1: now also U5.28 (PA8); no longer U5.30 (PC6)
- net ENC_A2: now also U5.30 (PC6); no longer U5.28 (PA8)
- net ENC_B1: now also U5.29 (PA9); no longer U5.31 (PC7)
- net ENC_B2: now also U5.31 (PC7); no longer U5.29 (PA9)
- net GPS_STATUS: no longer names the net of U5.20 (PB1)
- no-connect marks 23 -> 24
Other:
- note removed: "GPS Comms. Status"
- note removed: "GPS Status"
- moved on the sheet: D10, D3, D7, D8, D9, R20, R21, U5
