File: Precision Clock-backups/Precision Clock-2026-03-12_203712/User Inputs.kicad_sch (KiCad schematic)
At the start: 26 parts, among them SW1 PEC09-2320F-T0015, SW4 PEC09-2320F-T0015

Commit message: Routing
Parts:
- renumbered C26 to C28, C25 to C30, C27 to C31, C28 to C32, C30 to C33, C29 to C34, D16 to D12, D14 to D13, D15 to D14, D12 to D15, D17 to D16, D13 to D17, R7 to R10, R29 to R27, R32 to R28, R28 to R29, R35 to R31, R31 to R33, R10 to R5, R8 to R6, R9 to R7, R6 to R8, R11 to R9
Changed lines of the file:
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@@
 		(on_board yes)
 		(dnp no)
-		(property "Reference" "D13"
+		(property "Reference" "D17"
 			(at 245.618 95.504 90)
 			(effects
@@
 			(project "Precision Clock"
 				(path "/c9a8ff63-a0d1-4125-9dd1-40fb53daf536/47769572-a111-4c65-a7b3-f0883fcb5fca"
-					(reference "D13")
+					(reference "D17")
 					(unit 1)
 				)
@@
 		(dnp no)
 		(fields_autoplaced yes)
-		(property "Reference" "C30"
+		(property "Reference" "C33"
 			(at 219.71 71.1199 0)
 			(effects
@@
 			(project "Precision Clock"
 				(path "/c9a8ff63-a0d1-4125-9dd1-40fb53daf536/47769572-a111-4c65-a7b3-f0883fcb5fca"
-					(reference "C30")
+					(reference "C33")
 					(unit 1)
 				)
@@
 		(dnp no)
 		(fields_autoplaced yes)
-		(property "Reference" "R7"
+		(property "Reference" "R10"
 			(at 67.31 77.4701 0)
 			(effects
@@
 			(project "Precision Clock"
 				(path "/c9a8ff63-a0d1-4125-9dd1-40fb53daf536/47769572-a111-4c65-a7b3-f0883fcb5fca"
-					(reference "R7")
+					(reference "R10")
 					(unit 1)
 				)
@@
 		(on_board yes)
 		(dnp no)
-		(property "Reference" "D17"
+		(property "Reference" "D16"
 			(at 194.818 95.504 90)
 			(effects
@@
 			(project "Precision Clock"
 				(path "/c9a8ff63-a0d1-4125-9dd1-40fb53daf536/47769572-a111-4c65-a7b3-f0883fcb5fca"
-					(reference "D17")
+					(reference "D16")
 					(unit 1)
 				)
@@
 		(dnp no)
 		(fields_autoplaced yes)
-		(property "Reference" "C25"
+		(property "Reference" "C30"
 			(at 219.71 96.5199 0)
 			(effects
@@
 			(project ""
 				(path "/c9a8ff63-a0d1-4125-9dd1-40fb53daf536/47769572-a111-4c65-a7b3-f0883fcb5fca"
-					(reference "C25")
+					(reference "C30")
 					(unit 1)
 				)
@@
 		(on_board yes)
 		(dnp no)
-		(property "Reference" "D16"
+		(property "Reference" "D12"
 			(at 245.618 120.904 90)
 			(effects
@@
 			(project "Precision Clock"
 				(path "/c9a8ff63-a0d1-4125-9dd1-40fb53daf536/47769572-a111-4c65-a7b3-f0883fcb5fca"
-					(reference "D16")
+					(reference "D12")
 					(unit 1)
 				)
@@
 		(dnp no)
 		(fields_autoplaced yes)
-		(property "Reference" "R11"
+		(property "Reference" "R9"
 			(at 57.15 62.23 90)
 			(effects
@@
 			(project "Precision Clock"
 				(path "/c9a8ff63-a0d1-4125-9dd1-40fb53daf536/47769572-a111-4c65-a7b3-f0883fcb5fca"
-					(reference "R11")
+					(reference "R9")
 					(unit 1)
 				)
@@
 		(dnp no)
 		(fields_autoplaced yes)
-		(property "Reference" "R6"
+		(property "Reference" "R8"
 			(at 57.15 52.07 90)
 			(effects
@@
 			(project ""
 				(path "/c9a8ff63-a0d1-4125-9dd1-40fb53daf536/47769572-a111-4c65-a7b3-f0883fcb5fca"
-					(reference "R6")
+					(reference "R8")
 					(unit 1)
 				)
@@
 		(on_board yes)
 		(dnp no)
-		(property "Reference" "D12"
+		(property "Reference" "D15"
 			(at 194.818 120.904 90)
 			(effects
@@
 			(project "Precision Clock"
 				(path "/c9a8ff63-a0d1-4125-9dd1-40fb53daf536/47769572-a111-4c65-a7b3-f0883fcb5fca"
-					(reference "D12")
+					(reference "D15")
 					(unit 1)
 				)
@@
 		(dnp no)
 		(fields_autoplaced yes)
-		(property "Reference" "R8"
+		(property "Reference" "R6"
 			(at 120.65 54.61 90)
 			(effects
@@
 			(project "Precision Clock"
 				(path "/c9a8ff63-a0d1-4125-9dd1-40fb53daf536/47769572-a111-4c65-a7b3-f0883fcb5fca"
-					(reference "R8")
+					(reference "R6")
 					(unit 1)
 				)
@@
 		(dnp no)
 		(fields_autoplaced yes)
-		(property "Reference" "C27"
+		(property "Reference" "C31"
 			(at 270.51 71.1199 0)
 			(effects
@@
 			(project "Precision Clock"
 				(path "/c9a8ff63-a0d1-4125-9dd1-40fb53daf536/47769572-a111-4c65-a7b3-f0883fcb5fca"
-					(reference "C27")
+					(reference "C31")
 					(unit 1)
 				)
@@
 		(dnp no)
 		(fields_autoplaced yes)
-		(property "Reference" "R31"
+		(property "Reference" "R33"
 			(at 72.39 106.6799 0)
 			(effects
@@
 			(project "Precision Clock"
 				(path "/c9a8ff63-a0d1-4125-9dd1-40fb53daf536/47769572-a111-4c65-a7b3-f0883fcb5fca"
-					(reference "R31")
+					(reference "R33")
 					(unit 1)
 				)
@@
 		(dnp no)
 		(fields_autoplaced yes)
-		(property "Reference" "C29"
+		(property "Reference" "C34"
 			(at 219.71 121.9199 0)
 			(effects
@@
 			(project "Precision Clock"
 				(path "/c9a8ff63-a0d1-4125-9dd1-40fb53daf536/47769572-a111-4c65-a7b3-f0883fcb5fca"
-					(reference "C29")
+					(reference "C34")
 					(unit 1)
 				)
@@
 		(dnp no)
 		(fields_autoplaced yes)
-		(property "Reference" "R35"
+		(property "Reference" "R31"
 			(at 67.31 134.6201 0)
 			(effects
@@
 			(project "Precision Clock"
 				(path "/c9a8ff63-a0d1-4125-9dd1-40fb53daf536/47769572-a111-4c65-a7b3-f0883fcb5fca"
-					(reference "R35")
+					(reference "R31")
 					(unit 1)
 				)
@@
 		(dnp no)
 		(fields_autoplaced yes)
-		(property "Reference" "R9"
+		(property "Reference" "R7"
 			(at 113.03 49.5299 0)
 			(effects
@@
 			(project ""
 				(path "/c9a8ff63-a0d1-4125-9dd1-40fb53daf536/47769572-a111-4c65-a7b3-f0883fcb5fca"
-					(reference "R9")
+					(reference "R7")
 					(unit 1)
 				)
@@
 		(dnp no)
 		(fields_autoplaced yes)
-		(property "Reference" "C26"
+		(property "Reference" "C28"
 			(at 270.51 96.5199 0)
 			(effects
@@
 			(project "Precision Clock"
 				(path "/c9a8ff63-a0d1-4125-9dd1-40fb53daf536/47769572-a111-4c65-a7b3-f0883fcb5fca"
-					(reference "C26")
+					(reference "C28")
 					(unit 1)
 				)
@@
 		(dnp no)
 		(fields_autoplaced yes)
-		(property "Reference" "R32"
+		(property "Reference" "R28"
 			(at 57.15 109.22 90)
 			(effects
@@
 			(project "Precision Clock"
 				(path "/c9a8ff63-a0d1-4125-9dd1-40fb53daf536/47769572-a111-4c65-a7b3-f0883fcb5fca"
-					(reference "R32")
+					(reference "R28")
 					(unit 1)
 				)
@@
 		(dnp no)
 		(fields_autoplaced yes)
-		(property "Reference" "R29"
+		(property "Reference" "R27"
 			(at 57.15 119.38 90)
 			(effects
@@
 			(project "Precision Clock"
 				(path "/c9a8ff63-a0d1-4125-9dd1-40fb53daf536/47769572-a111-4c65-a7b3-f0883fcb5fca"
-					(reference "R29")
+					(reference "R27")
 					(unit 1)
 				)
@@
 		(dnp no)
 		(fields_autoplaced yes)
-		(property "Reference" "R10"
+		(property "Reference" "R5"
 			(at 72.39 49.5299 0)
 			(effects
@@
 			(project "Precision Clock"
 				(path "/c9a8ff63-a0d1-4125-9dd1-40fb53daf536/47769572-a111-4c65-a7b3-f0883fcb5fca"
-					(reference "R10")
+					(reference "R5")
 					(unit 1)
 				)
@@
 		(dnp no)
 		(fields_autoplaced yes)
-		(property "Reference" "C28"
+		(property "Reference" "C32"
 			(at 270.51 121.9199 0)
 			(effects
@@
 			(project "Precision Clock"
 				(path "/c9a8ff63-a0d1-4125-9dd1-40fb53daf536/47769572-a111-4c65-a7b3-f0883fcb5fca"
-					(reference "C28")
+					(reference "C32")
 					(unit 1)
 				)
@@
 		(on_board yes)
 		(dnp no)
-		(property "Reference" "D15"
+		(property "Reference" "D14"
 			(at 245.618 70.104 90)
 			(effects
@@
 			(project "Precision Clock"
 				(path "/c9a8ff63-a0d1-4125-9dd1-40fb53daf536/47769572-a111-4c65-a7b3-f0883fcb5fca"
-					(reference "D15")
+					(reference "D14")
 					(unit 1)
 				)
@@
 		(on_board yes)
 		(dnp no)
-		(property "Reference" "D14"
+		(property "Reference" "D13"
 			(at 194.818 70.104 90)
 			(effects
@@
 			(project "Precision Clock"
 				(path "/c9a8ff63-a0d1-4125-9dd1-40fb53daf536/47769572-a111-4c65-a7b3-f0883fcb5fca"
-					(reference "D14")
+					(reference "D13")
 					(unit 1)
 				)
@@
 		(dnp no)
 		(fields_autoplaced yes)
-		(property "Reference" "R28"
+		(property "Reference" "R29"
 			(at 120.65 111.76 90)
 			(effects
@@
 			(project "Precision Clock"
 				(path "/c9a8ff63-a0d1-4125-9dd1-40fb53daf536/47769572-a111-4c65-a7b3-f0883fcb5fca"
-					(reference "R28")
+					(reference "R29")
 					(unit 1)
 				)
