File: Precision Clock-backups/Precision Clock-2026-03-12_203712/_autosave-Precision Clock.kicad_pcb (KiCad board)
At the start: 4 copper layers, 220 x 55 mm, 146 parts, among them J1 50R SMA_Conn, J2 USB_C_Receptacle, J3 Conn_ST_STDC14, Q1 DMN3008SFG, Q2 DMN3008SFG, Q3 DMN3008SFG, Q4 TEPT5700, SW1 PEC09-2320F-T0015, SW2 B3U-1000P, SW3 B3U-1000P, SW4 PEC09-2320F-T0015, U1 MAX-M10S, U10 SA15-11SURKWA, U11 SA15-11SURKWA, U12 SA15-11SURKWA, U13 SA15-11SURKWA, U14 SA15-11SURKWA, U15 SA15-11SURKWA, U2 HDC1080, U3 W25Q32JVZP, U4 STM32G0B0CETx, U5 AP2127K-3.3, U6 TLC5926, U7 TLC5926, U8 TLC5926, U9 AP33771C, Y1 Q13MC14620002, Y2 ECS-TXO-2520MV

Commit message: Routing
Parts:
- removed D18: LED, precision_clock:LED_LiteON_LTST-C281KGKT
- removed the R42 at (224.0, 90.5)
- removed R43: 750R, Resistor_SMD:R_0402_1005Metric
- added TP10: SCL, TestPoint:TestPoint_Pad_D1.0mm, F.Cu at (232.0, 149.8)
- added TP4: OE, TestPoint:TestPoint_Pad_D1.0mm, F.Cu at (232.0, 137.6)
- added TP5: SDI, TestPoint:TestPoint_Pad_D1.0mm, F.Cu at (232.0, 140.6)
- added TP7: LE, TestPoint:TestPoint_Pad_D1.0mm, F.Cu at (232.0, 143.7)
- added TP9: SDO, TestPoint:TestPoint_Pad_D1.0mm, F.Cu at (232.0, 146.7)
- moved R40 3.07 mm to (200.4, 106.0)
- moved TP17 1.80 mm to (78.5, 103.0)
- moved D10 1.25 mm to (212.8, 90.5)
- moved R20 1.21 mm to (215.4, 91.1)
- moved R21 1.21 mm to (215.4, 89.9)
- renumbered C13 to C11, C8 to C12, C6 to C13, C15 to C16, C20 to C17, C17 to C18, C18 to C19, C16 to C20, C19 to C21, C14 to C24, C21 to C25, C23 to C26, C22 to C27, C26 to C28, C24 to C29, C25 to C30, C27 to C31, C28 to C32, C30 to C33, C29 to C34, C31 to C35, C35 to C36, C32 to C37, C34 to C38, C36 to C39, C33 to C40, C37 to C41, C38 to C42, C39 to C43, C40 to C44, C41 to C45, C42 to C46, C7 to C6, C12 to C7, C9 to C8, C11 to C9, D2 to D1, D11 to D10, D10 to D11, D16 to D12, D14 to D13, D15 to D14, D12 to D15, D17 to D16, D13 to D17, D1 to D2, D6 to D5, D9 to D6, D5 to D7, D7 to D8, D8 to D9, JP2 to JP1, JP1 to JP2, R7 to R10, R14 to R11, R16 to R12, R12 to R13, R13 to R14, R17 to R16, R18 to R17, R21 to R18, R41 to R19, R22 to R20, R23 to R21, R20 to R22, R25 to R23, R26 to R24, R27 to R25, R33 to R26, R29 to R27, R32 to R28, R28 to R29, R35 to R31, R36 to R32, R31 to R33, R37 to R34, R34 to R35, R39 to R36, R38 to R37, R40 to R38, R5 to R4, R19 to R40, R24 to R41, R4 to R42, R10 to R5, R8 to R6, R9 to R7, R6 to R8, R11 to R9, TP2 to TP1, TP4 to TP17, TP1 to TP2, U3 to U16, U5 to U4, U4 to U5
Connections:
- net /MCU/BT0/SWDCLK renamed /MCU/BT0/SWCLK
- net /MCU/SWDIO renamed /MCU/SWIO
- U5 pad 15: /GPS/GPS.TX -> /GPS/GPS.RX
- U5 pad 16: /GPS/GPS.RX -> /GPS/GPS.TX
- U5 pad 20: /MCU/GPS_STATUS -> unconnected-(U5-PB1-Pad20)
- U5 pad 28: /MCU/ENC_A2 -> unconnected-(U5-PA8-Pad28)
- U5 pad 29: /MCU/ENC_B2 -> /MCU/ENC_A1
- U5 pad 30: /MCU/ENC_A1 -> /MCU/ENC_A2
- U5 pad 31: /MCU/ENC_B1 -> /MCU/ENC_B2
- U5 pad 32: unconnected-(U4-PA10-Pad32) -> /MCU/ENC_B1
- U5 pad 39: /Clock Display/LE -> unconnected-(U5-PD1-Pad39)
- U5 pad 45: unconnected-(U4-PB6-Pad45) -> /Clock Display/LE
Routing:
- net /MCU/GPS_STATUS: track 25.8 -> 0.00 mm, vias 2 -> 0
- net /MCU/ENC_A1: track 165.8 -> 173.0 mm
- net /Clock Display/LE: track 84.2 -> 89.2 mm
- net /Buzzer/BZ: track 160.5 -> 156.1 mm
- net /MCU/SPI_CLK: track 5.55 -> 2.19 mm
- net /Clock Display/SCL: track 74.9 -> 78.3 mm
- net Net-(D18-K): track 2.77 -> 0.00 mm
- net /MCU/ENC_B1: track 162.5 -> 164.9 mm
- net /MCU/BT0/SWCLK: track 59.8 -> 61.6 mm
- net /MCU/ENC_A2: track 163.1 -> 161.5 mm
- net /MCU/ENC_B2: track 157.8 -> 156.4 mm
- net /GPS/GPS.RX: track 38.8 -> 38.2 mm, vias 0 -> 2
- net /GPS/GPS.TP: track 36.3 -> 35.7 mm
- net /GPS/GPS.TX: track 37.8 -> 38.5 mm
- net MCU_RTC: vias 0 -> 1
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Other:
- board text added: "QSPI 133MHz 32MB"
- board text added: "STM32U575RGT6"
- board text removed: "GPS_OK"
- board text removed: "SPI FLASH 32MB"
- board text removed: "STM32G0B0CET6"
