File: Precision Clock-backups/Precision Clock-2026-03-12_203712/gps.kicad_sch (KiCad schematic)
At the start: 8 parts, among them J1 50R SMA_Conn, U1 MAX-M10S

Commit message: Routing
Parts:
- renumbered C11 to C9
Changed lines of the file:
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@@
 		(dnp no)
 		(fields_autoplaced yes)
-		(property "Reference" "C11"
+		(property "Reference" "C9"
 			(at 123.19 76.1999 0)
 			(effects
@@
 			(project "Precision Clock"
 				(path "/c9a8ff63-a0d1-4125-9dd1-40fb53daf536/adbcdd61-c016-4293-925d-555ee31f0e50"
-					(reference "C11")
+					(reference "C9")
 					(unit 1)
 				)
