File: Precision Clock-backups/Precision Clock-2026-03-12_203712/Ambient Light Sensor.kicad_sch (KiCad schematic)
At the start: 0 parts

Commit message: Verification
Parts:
- added C4: 100n, Capacitor_SMD:C_0402_1005Metric, symbol Device:C
- added Q4: TEPT5700, LED_THT:LED_D5.0mm_Clear, symbol Sensor_Optical:TEPT4400
- added R11: 510R, Resistor_SMD:R_0402_1005Metric, symbol Device:R
- added R13: 10K, Resistor_SMD:R_0402_1005Metric, symbol Device:R
- added TP3: ALS, TestPoint:TestPoint_Pad_D1.0mm, symbol Connector:TestPoint
Connections:
- new net: Q4.1 (C), R11.1, R13.2
- new net +3.3V: C4.1, R13.1
- new net ALS: R11.2, TP3.1
- new net GND: C4.2, Q4.2 (E)
Other:
- note added: "Ambient Light Sensor"
- company: (none) -> TJ71PL
- title: (none) -> Ambient Light Sensor
