File: Precision Clock-backups/Precision Clock-2026-03-12_203712/Power.kicad_sch (KiCad schematic)
At the start: 0 parts

Commit message: Verification
Parts:
- added BT1: CR2032, precision_clock:Battery_holder_CR2032_SMD, symbol Device:Battery_Cell
- added C10, C12, C40, C7: 10u, Capacitor_SMD:C_0603_1608Metric, symbol Device:C
- added C11, C13, C39: 100n, Capacitor_SMD:C_0402_1005Metric, symbol Device:C
- added C35, C38: 10n, Capacitor_SMD:C_0402_1005Metric, symbol Device:C
- added C37, C42, C6: 1u, Capacitor_SMD:C_0402_1005Metric, symbol Device:C
- added D11, D2, D4: LED, precision_clock:LED_LiteON_LTST-C281KGKT, symbol Device:LED
- added JP1: GPS_BCKP, Jumper:SolderJumper-2_P1.3mm_Open_TrianglePad1.0x1.5mm, symbol Jumper:SolderJumper_2_Open
- added JP2: MCU_RTC, Jumper:SolderJumper-2_P1.3mm_Open_TrianglePad1.0x1.5mm, symbol Jumper:SolderJumper_2_Open
- added Q1, Q2: DMN3008SFG, Package_SON:Diodes_PowerDI3333-8, symbol Transistor_FET:DMN3008SFG
- added R12, R14, R38: 5.1K, Resistor_SMD:R_0402_1005Metric, symbol Device:R
- added R15, R18, R19, R22: 750R, Resistor_SMD:R_0402_1005Metric, symbol Device:R
- added R17: 5mR, Resistor_SMD:R_0805_2012Metric, symbol Device:R
- added R36: 39K, Resistor_SMD:R_0402_1005Metric, symbol Device:R
- added R37: 100K, Resistor_SMD:R_0402_1005Metric, symbol Device:R
- added U4: AP2127K-3.3, Package_TO_SOT_SMD:SOT-23-5, symbol Regulator_Linear:AP2127K-3.3
- added U9: AP33771C, precision_clock:W-DFN3030-14 (Type A1) Diodes, symbol precision_clock:AP33771C
Connections:
- new net: C12.1, C7.1, Q1.1 (S), Q1.2 (S), Q1.3 (S), R17.2, U9.3 (VCC)
- new net: Q1.4 (G), Q2.4 (G), R38.2
- new net: Q1.5 (D), Q2.5 (D)
- new net: C6.1, U9.14 (V5V)
- new net: D4.1 (K), R18.1
- new net: R38.1, U9.2 (PWREN)
- new net: C38.1, R37.1, U9.8 (VSEL)
- new net: C35.1, R36.1, U9.9 (ISEL)
- new net: D2.1 (K), R15.1
- new net: D11.1 (K), R19.1, R22.1
- new net +3.3V: C42.1, D11.2 (A), U4.5 (VOUT)
- new net +BATT: BT1.1 (+), JP1.1 (A), JP2.1 (A)
- new net CC1: R12.1, U9.11 (CC1)
- new net CC2: R14.1, U9.10 (CC2)
- new net GND: BT1.2 (-), C10.2, C11.2, C12.2, C13.2, C35.2, C37.2, C38.2, C39.2, C40.2, C42.2, C6.2, C7.2, R12.2, R14.2, R15.2, R18.2, R19.2, R22.2, R36.2, R37.2, U4.2 (GND), U9.15 (EPAD), U9.5 (GND)
- new net GPS_BCKP: JP1.2 (B)
- new net LED: D2.2 (A), U9.7 (LED)
- new net MCU_RTC: JP2.2 (B)
- new net USB_D+: U9.13 (DP)
- new net USB_D-: U9.12 (DN)
- new net VBUS: C10.1, C11.1, C39.1, R17.1, U9.4 (ISENP)
- new net VD: C13.1, C37.1, C40.1, D4.2 (A), Q2.1 (S), Q2.2 (S), Q2.3 (S), U4.1 (VIN), U4.3 (EN), U9.1 (VOUT)
- no-connect marks 0 -> 1
Other:
- note added: "3.3V LDO"
- note added: "3.3V OK"
- note added: "3.3V Rail"
- note added: "Backup Battery"
- note added: "Backup Battery Voltage Rail"
- note added: "Display Voltage OK"
- note added: "Display Voltage Rail"
- note added: "LED Indications of System States"
- note added: "PD System State"
- note added: "Power Status Indicators"
- note added: "USB PD Adapters or Power Banks capable of providing 3A@5V should be used."
- note added: "USB PD3.1 Sink"
- company: (none) -> TJ71PL
- title: (none) -> Power Negotiation & Regulation
