File: electronics/Precision Clock.kicad_pcb (KiCad board)
At the start: 4 copper layers, 220 x 55 mm, 153 parts, among them J1 50R SMA_Conn, J2 USB_C_Receptacle, J3 Conn_ST_STDC14, Q1 DMN3008SFG, Q2 DMN3008SFG, Q3 DMN3008SFG, Q4 TEPT5700, SW1 PEC09-2320F-T0015, SW2 B3U-1000P, SW3 B3U-1000P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

Commit message: In Production
Other:
- board text added: "GNSS SYNCRONIZED PRECISION CLOCK ΔT±0.0001s TJ71PL"
- board text added: "ΔT ±1us Internal"
- board text removed: "GNSS SYNCRONIZED PRECISION CLOCK ΔT±0.00001s TJ71PL"
- board text removed: "ΔT ±0.2us Internal"
